File: cad/mini32.brd (EAGLE design)
At the start: 63 x 35 mm, 54 parts, among them CN1 MICROSDPLAIN, J1 HEADER-5X1, Q1 MOSFETSOT-23, Q2 MOSFET-P, SW2 SWITCHKMR211, SW3 SWITCHKMR211, U1 STM32F411/48, U2 MPU-9150, U3 MCP73831/OT, U4 MCP1824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

Commit message: replace charger
Parts:
- removed D2: DIODESOD-323, jaw:SOD-323
- removed Q2: MOSFET-P, jaw:SOT-23
- removed R2: 100k, jaw:SMD0603
- added C17: (no value), jaw:SMD0603
- R1: value 10k -> (none)
- U3: value MCP73831/OT -> ADP5062; device adafruit:SOT23-5L -> jaw:LGA20P
- moved U3 2.84 mm to (4.00, 23.0), turned to 90 degrees
- moved R1 2.59 mm to (3.20, 18.0), turned to 270 degrees
Connections:
- removed net N$1: R1.2, U3.5
- new net N$5: C17.2, U3.19
- new net N$6: R1.1, U3.18
- net BATSTAT: no longer U3.1
- net GND: now also C17.1, R1.2, U3.20, U3.3, U3.PAD; no longer R1.1, R2.1, U3.2
- net I2CCL: now also U3.1
- net I2CDA: now also U3.17
- net VBAT: now also U3.12, U3.13, U3.14, U3.4; no longer Q2.3, U3.3
- net VP: now also U3.10, U3.11, U3.2, U3.5, U3.9; no longer D2.C, Q2.2
- net VUSB: now also U3.6, U3.7, U3.8; no longer D2.A, Q2.1, R2.2, U3.4
Routing:
- net I2CDA: track 45.7 -> 92.6 mm, vias 3 -> 4
- net I2CCL: track 46.5 -> 90.8 mm, vias 1 -> 2
- net BATSTAT: track 36.7 -> 22.1 mm, vias 2 -> 1
- net VBAT: track 20.7 -> 33.1 mm, vias 0 -> 2
- net VP: track 8.52 -> 16.9 mm, vias 0 -> 4
- net VUSB: track 92.2 -> 84.0 mm, vias 3 -> 2
- net GND: track 107.8 -> 110.6 mm, vias 23 -> 24
- net N$5: track 0.00 -> 2.51 mm
- net N$6: track 0.00 -> 2.13 mm
- net N$1: track 1.75 -> 0.00 mm
- net N$12: track 9.34 -> 8.40 mm
- net N$16: track 9.26 -> 8.40 mm
- added copper zone on layer 16, net GND
- added copper zone on layer 2, net VCC
- added copper zone on layer 2, net VP

Commit message: ok
Parts:
- removed C6, C7: (no value), jaw:SMD0603
- removed U$1: (no value), adafruit:CR2032-SMD
- added B1: BATTERY-CR2016, jaw:CR1216
- added U$4: ROBOTMAN-LOGO, jaw:ROBOTMAN-LOGO
- C12: value (none) -> 0.1u
- C13: value (none) -> 2.2n
- C14: value (none) -> .1u
- C17: value (none) -> 10n
- C8, C9: value (none) -> 5p
- R1: value (none) -> 10k
- R8: value (none) -> 470
- X1: value XTAL32X15 -> 12MHz; device jaw:XTAL-32X15 -> jaw:RESONATOR-CSTCE
- X2: value XTAL32X15 -> 32k768
- moved C17 0.50 mm to (5.50, 18.0)
- moved R1 0.50 mm to (3.70, 18.0)
- moved CN3 0.30 mm to (3.70, 11.0)
- moved X1 0.10 mm to (26.5, 17.7)
Connections:
- removed net N$29: U1.P40
- new net IMUINT: U1.P40, U2.12
- net BATSTAT: now also U3.16
- net GND: now also B1.MINUS, X1.2; no longer C6.1, C7.1, U$1.+$2
- net N$12: now also X1.1; no longer C6.2, X1.P$1
- net N$13: now also X1.3; no longer C7.2, X1.P$2
- net N$21: now also B1.PLUS1, B1.PLUS2; no longer U$1.-
Routing:
- net IMUINT: track 0.00 -> 24.7 mm, vias 0 -> 2
- net N$21: track 5.36 -> 27.3 mm, vias 1 -> 3
- net BATSTAT: track 22.1 -> 39.6 mm, vias 1 -> 2
- net N$13: track 9.03 -> 4.20 mm
- net BOOT0: track 32.7 -> 35.2 mm, vias 3 -> 4
- net VP: track 16.9 -> 19.0 mm, vias 4 -> 5
- net NRST: track 130.0 -> 128.3 mm
- net N$12: track 8.40 -> 7.04 mm
- net VCC: track 69.5 -> 70.7 mm
- net GND: track 110.6 -> 111.8 mm, vias 24 -> 72
- net I2CDA: track 92.6 -> 93.3 mm
- net N$15: track 8.99 -> 9.75 mm
- net VBAT: track 33.1 -> 33.8 mm
- net I2CCL: track 90.8 -> 90.1 mm
- added copper zone on layer 1, net GND
- added copper zone on layer 15, net GND
Other:
- outline, holes or cut-outs redrawn
- board text added: "+"
- board text added: "BT0"
- board text added: "CK"
- board text added: "IO"
- board text added: "JAW 2015-03"
- board text added: "JAW mini32/11"
- board text added: "NRST"
- board text added: "Pb"
- board text added: "RST"
- board text added: "SD card"
- board text added: "SWD"
- board text added: "V"
- board text added: "VP"
- board text added: "Vu"
- board text added: "battery - CR1216"
- board text added: "display"
- board text added: "mini32/11 Rev. 0"
- board text added: "www.tcp4me.com"

Commit message: lsm303d
Parts:
- C12: value 0.1u -> 4.7u
- C13: value 2.2n -> .22u
- U2: value MPU-9150 -> LSM303D; device jaw:LGA24 -> jaw:LGA16A
- moved C12 8.30 mm to (35.5, 30.8), turned to 90 degrees
- moved C14 7.30 mm to (42.5, 31.0)
- moved U2 0.71 mm to (39.0, 30.5), turned to 0 degrees
- moved C13 0.40 mm to (34.5, 27.7), turned to 0 degrees
Connections:
- new net N$1: C12.1, U2.15
- net GND: now also U2.10, U2.12, U2.13, U2.16, U2.5, U2.7; no longer C13.2, U2.1, U2.11, U2.15, U2.17, U2.18, U2.9
- net I2CCL: now also U2.4; no longer U2.23
- net I2CDA: now also U2.6; no longer U2.24
- net IMUINT: now also U2.11; no longer U2.12
- net N$2: now also C13.2, U2.3; no longer C12.1, U2.10
- net N$4: now also U2.2; no longer U2.20
- net VCC: now also U2.1, U2.14; no longer U2.13, U2.3
Routing:
- net GND: track 111.8 -> 101.8 mm
- net I2CDA: track 93.3 -> 96.0 mm
- net N$1: track 0.00 -> 2.31 mm
- net N$4: track 5.37 -> 7.66 mm
- net IMUINT: track 24.7 -> 23.0 mm, vias 2 -> 0
- net VCC: track 70.7 -> 69.2 mm, vias 14 -> 16
- net N$2: track 7.09 -> 5.94 mm
- net I2CCL: track 90.1 -> 91.0 mm

Commit message: max17048
Parts:
- added U5: MAX17048, jaw:TDFN8EP
Connections:
- new net N$22: U5.5
- net GND: now also U5.1, U5.4, U5.6, U5.PAD
- net I2CCL: now also U5.7
- net I2CDA: now also U5.8
- net VBAT: now also U5.3
Routing:
- net I2CCL: track 91.0 -> 112.3 mm, vias 2 -> 3
- net I2CDA: track 96.0 -> 111.9 mm, vias 4 -> 5
- net N$21: track 27.3 -> 34.3 mm
- net GND: track 101.8 -> 108.5 mm, vias 72 -> 74
- net VBAT: track 33.8 -> 39.9 mm

Commit message: embiggen connectors
Parts:
- removed CN6: (no value), jaw:HEADER-2X04
- added CONN1: HEADER-5X2-PTH, jaw:HEADER-5X2-PTH
- added LOGO1: OSHW-LOGOM, Sparkfun-Aesthetics:OSHW-LOGO-M
- added U$1: ROBOTMAN-LOGO, jaw:ROBOTMAN-LOGO
- JP1: value (none) -> HEADER-21X1; device adafruit:1X20 -> jaw:HEADER-21X1-PTH
- moved C16 3.10 mm to (56.0, 21.5)
- moved R18 3.10 mm to (52.5, 21.5)
- moved CN1 3.00 mm to (57.0, 13.5)
- moved U$2 3.00 mm to (59.0, 32.5)
- moved USB1 3.00 mm to (63.0, 25.0)
- moved U$3 0.50 mm to (11.0, 8.00)
- moved JP1 0.13 mm to (26.7, 2.03)
Connections:
- net BOOT0: now also JP1.15
- net DPYCS: now also CONN1.7; no longer CN6.7
- net DPYDC: now also CONN1.6; no longer CN6.6
- net GND: now also CONN1.8; no longer CN6.8
- net I2CCL: now also CONN1.9, JP1.17; no longer JP1.15
- net I2CDA: now also CONN1.10, JP1.18; no longer JP1.16
- net NRST: now also CONN1.2, JP1.16; no longer CN6.2, JP1.17
- net SPIMISO: now also CONN1.3, JP1.21; no longer CN6.3, JP1.20
- net SPIMOSI: now also CONN1.5, JP1.20; no longer CN6.5, JP1.19
- net SPISCK: now also CONN1.4, JP1.19; no longer CN6.4, JP1.18
- net VCC: now also CONN1.1; no longer CN6.1
Routing:
- net GND: track 108.5 -> 139.0 mm, vias 74 -> 76
- net BOOT0: track 35.2 -> 55.5 mm, vias 4 -> 6
- net I2CCL: track 112.3 -> 126.9 mm
- net I2CDA: track 111.9 -> 123.6 mm
- net NRST: track 128.2 -> 139.1 mm
- net SPIMOSI: track 44.7 -> 52.5 mm
- net SPIMISO: track 42.0 -> 46.2 mm
- net IOCARD: track 18.5 -> 21.6 mm
- net DPYDC: track 29.9 -> 32.9 mm
- net SDCS: track 21.6 -> 24.6 mm
- net N$8: track 7.94 -> 10.9 mm
- net N$7: track 7.93 -> 10.9 mm
- net N$3: track 4.70 -> 7.70 mm
- net TX: track 28.1 -> 30.1 mm
- net SPISCK: track 46.4 -> 48.0 mm
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Other:
- board size 63 x 35 mm -> 66 x 35 mm
- board text added: "X"
- board text added: "Y"
- board text added: "Z"
- board text added: "www.791RL.com"
- board text removed: "nRST"
- board text removed: "www.tcp4me.com"

Commit message: tweak
Parts:
- added R2: 100, jaw:SMD0603
Connections:
- new net N$9: Q1.1, R2.2
- net IOB9: now also R2.1; no longer Q1.1
Routing:
- net IOB9: track 18.1 -> 11.7 mm
- net N$9: track 0.00 -> 5.83 mm
- net DPYCS: track 25.8 -> 25.6 mm, vias 1 -> 0

Commit message: 8pin dpy
Parts:
- removed CONN1: HEADER-5X2-PTH, jaw:HEADER-5X2-PTH
- added CN6: (no value), jaw:HEADER-2X04
- moved C16 2.00 mm to (54.0, 21.5)
- moved CN1 2.00 mm to (55.0, 13.5)
- moved R18 2.00 mm to (50.5, 21.5)
- moved U$2 2.00 mm to (57.0, 32.5)
- moved USB1 2.00 mm to (61.0, 25.0)
- moved U$1 0.14 mm to (44.0, 18.6)
Connections:
- net DPYCS: now also CN6.7; no longer CONN1.7
- net DPYDC: now also CN6.6; no longer CONN1.6
- net GND: now also CN6.8; no longer CONN1.8
- net I2CCL: no longer CONN1.9
- net I2CDA: no longer CONN1.10
- net NRST: now also CN6.2; no longer CONN1.2
- net SPIMISO: now also CN6.3; no longer CONN1.3
- net SPIMOSI: now also CN6.5; no longer CONN1.5
- net SPISCK: now also CN6.4; no longer CONN1.4
- net VCC: now also CN6.1; no longer CONN1.1
Routing:
- net I2CCL: track 126.9 -> 110.6 mm
- net I2CDA: track 123.6 -> 110.2 mm
- net GND: track 139.0 -> 130.0 mm, vias 76 -> 75
- net NRST: track 139.1 -> 131.9 mm
- net SPIMISO: track 46.2 -> 43.0 mm
- net BOOT0: track 55.5 -> 52.6 mm, vias 6 -> 5
- net SDCS: track 24.6 -> 22.6 mm
- net N$8: track 10.9 -> 8.94 mm
- net N$7: track 10.9 -> 8.93 mm
- net N$3: track 7.70 -> 5.70 mm
- net IOCARD: track 21.6 -> 19.6 mm
- net DPYDC: track 32.9 -> 31.2 mm
- net DPYCS: track 25.6 -> 24.4 mm
- net SPIMOSI: track 52.5 -> 52.2 mm, vias 2 -> 1
Other:
- board size 66 x 35 mm -> 64 x 35 mm
- board text added: "LiPo"

Commit message: tweak
Routing:
- net GND: track 130.0 -> 132.2 mm, vias 75 -> 74
Other:
- board text added: "USB"
