File: cad/mini32.sch (EAGLE design)
At the start: 55 parts, among them CN1 MICROSDPLAIN, J1 HEADER-5X1, Q1 MOSFETSOT-23, SW2 SWITCHKMR211, SW3 SWITCHKMR211, U1 STM32F411/48, U2 LSM303D, U3 ADP5062, U4 MCP1824, U5 MAX17048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

Commit message: fix vreg
Connections:
- net GND: no longer U4.NSHTDN
- net VP: now also U4.NSHTDN
Changed lines of the file:
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@@
 <layer number="113" name="IDFDebug" color="4" fill="1" visible="yes" active="yes"/>
 <layer number="116" name="Patch_BOT" color="7" fill="1" visible="yes" active="yes"/>
+<layer number="118" name="Rect_Pads" color="7" fill="1" visible="no" active="no"/>
 <layer number="121" name="_tsilk" color="7" fill="1" visible="yes" active="yes"/>
 <layer number="122" name="_bsilk" color="7" fill="1" visible="yes" active="yes"/>
@@
 <layer number="230" name="230bmp" color="7" fill="1" visible="yes" active="yes"/>
 <layer number="231" name="231bmp" color="7" fill="1" visible="yes" active="yes"/>
+<layer number="232" name="Eagle3D_PG2" color="7" fill="1" visible="no" active="no"/>
+<layer number="233" name="Eagle3D_PG3" color="7" fill="1" visible="no" active="no"/>
 <layer number="248" name="Housing" color="7" fill="1" visible="yes" active="yes"/>
 <layer number="249" name="Edge" color="7" fill="1" visible="yes" active="yes"/>
@@
 </segment>
 <segment>
-<pinref part="U4" gate="G$1" pin="NSHTDN"/>
 <pinref part="U4" gate="G$1" pin="GND"/>
-<wire x1="93.98" y1="55.88" x2="93.98" y2="48.26" width="0.1524" layer="91"/>
 <wire x1="93.98" y1="48.26" x2="109.22" y2="48.26" width="0.1524" layer="91"/>
 <pinref part="GND3" gate="G$1" pin="GND"/>
@@
 <wire x1="88.9" y1="50.8" x2="88.9" y2="48.26" width="0.1524" layer="91"/>
 <wire x1="88.9" y1="48.26" x2="93.98" y2="48.26" width="0.1524" layer="91"/>
-<junction x="93.98" y="48.26"/>
 <pinref part="C5" gate="G$1" pin="P$2"/>
 <wire x1="154.94" y1="50.8" x2="154.94" y2="48.26" width="0.1524" layer="91"/>
@@
 <pinref part="C1" gate="G$1" pin="P$1"/>
 <pinref part="U4" gate="G$1" pin="VIN"/>
-<wire x1="88.9" y1="58.42" x2="93.98" y2="58.42" width="0.1524" layer="91"/>
+<wire x1="88.9" y1="58.42" x2="91.44" y2="58.42" width="0.1524" layer="91"/>
 <junction x="88.9" y="58.42"/>
+<wire x1="91.44" y1="58.42" x2="93.98" y2="58.42" width="0.1524" layer="91"/>
 <wire x1="81.28" y1="58.42" x2="88.9" y2="58.42" width="0.1524" layer="91"/>
 <wire x1="81.28" y1="58.42" x2="81.28" y2="66.04" width="0.1524" layer="91"/>
@@
 <wire x1="53.34" y1="58.42" x2="81.28" y2="58.42" width="0.1524" layer="91"/>
 <junction x="81.28" y="58.42"/>
-</segment>
-<segment>
+<pinref part="U4" gate="G$1" pin="NSHTDN"/>
+<wire x1="93.98" y1="55.88" x2="91.44" y2="55.88" width="0.1524" layer="91"/>
+<wire x1="91.44" y1="55.88" x2="91.44" y2="58.42" width="0.1524" layer="91"/>
+<junction x="91.44" y="58.42"/>
+</segment>
+<segment>

Commit message: silk text
Parts:
- U$1, U$4: value ROBOTMAN-LOGO -> ROBOTMAN-LOGO2; device jaw:ROBOTMAN-LOGO -> jaw:ROBOTMAN-LOGO2
Changed lines of the file:
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@@
 <part name="GND11" library="jaw" deviceset="PWR-GND" device=""/>
 <part name="GND21" library="jaw" deviceset="PWR-GND" device=""/>
-<part name="U$4" library="jaw" deviceset="ROBOTMAN-LOGO" device=""/>
+<part name="U$4" library="jaw" deviceset="ROBOTMAN-LOGO" device="2" value="ROBOTMAN-LOGO2"/>
 <part name="B1" library="jaw" deviceset="BATTERY" device="-CR2016"/>
 <part name="X1" library="jaw" deviceset="RESONATOR" device="CTCE" value="12MHz"/>
@@
 <part name="U5" library="jaw" deviceset="MAX17048" device=""/>
 <part name="LOGO1" library="Sparkfun-Aesthetics" deviceset="OSHW-LOGO" device="M"/>
-<part name="U$1" library="jaw" deviceset="ROBOTMAN-LOGO" device=""/>
+<part name="U$1" library="jaw" deviceset="ROBOTMAN-LOGO" device="2" value="ROBOTMAN-LOGO2"/>
 <part name="R2" library="jaw" deviceset="R" device="0603" value="100"/>
 <part name="CN6" library="jaw" deviceset="HEADER-2X4" device=""/>

Commit message: add p-mosfet on sd+dpy power
Parts:
- added C6: 1u, jaw:C0603
- added Q2: DMP2035U-7, jaw:MOSFET-P
- L1: value 40u -> 10u
- LED1: value LED -> white
- Q1: value MOSFETSOT-23 -> IRLML6344TRPBF
- R18: value 10k -> 100k
Connections:
- new net NPWREN: Q2.G, U1.PB5
- new net VCCE: C16.P$1, C6.P$1, CN1.SW1, CN1.VCC, CN6.P$1, Q2.D
- net BATSTAT: no longer U1.PB5
- net GND: now also C6.P$2
- net VCC: now also Q2.S; no longer C16.P$1, CN1.SW1, CN1.VCC, CN6.P$1
Other:
- note added: "to reduce leakage current thru dpy + sd card while off"
Changed lines of the file:
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@@
 <setting verticaltext="up"/>
 </settings>
-<grid distance="0.1" unitdist="inch" unit="inch" style="lines" multiple="1" display="no" altdistance="0.01" altunitdist="inch" altunit="inch"/>
+<grid distance="0.1" unitdist="inch" unit="inch" style="lines" multiple="1" display="yes" altdistance="0.01" altunitdist="inch" altunit="inch"/>
 <layers>
 <layer number="1" name="Top" color="4" fill="1" visible="no" active="no"/>
@@
 <part name="VCC1" library="jaw" deviceset="PWR-VCC" device=""/>
 <part name="VCCA1" library="jaw" deviceset="PWR-VCCA" device=""/>
-<part name="L1" library="jaw" deviceset="L" device="SMD0603" value="40u"/>
+<part name="L1" library="jaw" deviceset="L" device="SMD0603" value="10u"/>
 <part name="C5" library="jaw" deviceset="C" device="0603" value="10u"/>
 <part name="X2" library="jaw" deviceset="XTAL" device="32X15" value="32k768"/>
@@
 <part name="R6" library="jaw" deviceset="R" device="0603" value="22"/>
 <part name="R7" library="jaw" deviceset="R" device="0603" value="22"/>
-<part name="LED1" library="jaw" deviceset="LED" device=""/>
+<part name="LED1" library="jaw" deviceset="LED" device="" value="white"/>
 <part name="R8" library="jaw" deviceset="R" device="0603" value="470"/>
 <part name="GND9" library="jaw" deviceset="PWR-GND" device=""/>
@@
 <part name="VCC3" library="jaw" deviceset="PWR-VCC" device=""/>
 <part name="GND10" library="jaw" deviceset="PWR-GND" device=""/>
-<part name="Q1" library="jaw" deviceset="MOSFET" device="SOT-23"/>
+<part name="Q1" library="jaw" deviceset="MOSFET" device="SOT-23" value="IRLML6344TRPBF"/>
 <part name="CN1" library="jaw" deviceset="MICROSD" device="PLAIN"/>
 <part name="GND22" library="jaw" deviceset="PWR-GND" device=""/>
-<part name="VCC18" library="jaw" deviceset="PWR-VCC" device=""/>
 <part name="C16" library="jaw" deviceset="C" device="0603" value="4.7u"/>
-<part name="VCC19" library="jaw" deviceset="PWR-VCC" device=""/>
 <part name="GND23" library="jaw" deviceset="PWR-GND" device=""/>
-<part name="R18" library="jaw" deviceset="R" device="0603" value="10k"/>
+<part name="R18" library="jaw" deviceset="R" device="0603" value="100k"/>
 <part name="GND13" library="jaw" deviceset="PWR-GND" device=""/>
 <part name="U$2" library="adafruit" deviceset="FIDUCIAL" device=""/>
@@
 <part name="CN6" library="jaw" deviceset="HEADER-2X4" device=""/>
 <part name="GND24" library="jaw" deviceset="PWR-GND" device=""/>
-<part name="VCC20" library="jaw" deviceset="PWR-VCC" device=""/>
+<part name="Q2" library="jaw" deviceset="MOSFET-P" device="" value="DMP2035U-7"/>
+<part name="VCC5" library="jaw" deviceset="PWR-VCC" device=""/>
+<part name="VCCE1" library="jaw" deviceset="PWR-VCCE" device=""/>
+<part name="VCCE2" library="jaw" deviceset="PWR-VCCE" device=""/>
+<part name="VCCE3" library="jaw" deviceset="PWR-VCCE" device=""/>
+<part name="VCCE4" library="jaw" deviceset="PWR-VCCE" device=""/>
+<part name="C6" library="jaw" deviceset="C" device="0603" value="1u"/>
 </parts>
 <sheets>
@@
 <plain>
 <text x="198.12" y="88.9" size="3.81" layer="97">SD CARD</text>
-<text x="241.3" y="50.8" size="3.81" layer="97">display</text>
+<text x="248.92" y="58.42" size="3.81" layer="97">display</text>
 <text x="241.3" y="182.88" size="3.81" layer="97">JTAG/SWD</text>
+<text x="137.16" y="88.9" size="1.27" layer="97">to reduce leakage current
+thru dpy + sd card while off</text>
 </plain>
 <instances>
@@
 <instance part="CN1" gate="G$1" x="205.74" y="73.66"/>
 <instance part="GND22" gate="G$1" x="177.8" y="60.96"/>
-<instance part="VCC18" gate="G$1" x="177.8" y="68.58"/>
 <instance part="C16" gate="G$1" x="220.98" y="73.66"/>
-<instance part="VCC19" gate="G$1" x="220.98" y="81.28"/>
 <instance part="GND23" gate="G$1" x="220.98" y="68.58"/>
 <instance part="R18" gate="G$1" x="228.6" y="58.42"/>
@@
 <instance part="CN6" gate="A" x="251.46" y="71.12"/>
 <instance part="GND24" gate="G$1" x="264.16" y="66.04"/>
-<instance part="VCC20" gate="G$1" x="236.22" y="78.74"/>
+<instance part="Q2" gate="G$1" x="147.32" y="76.2" rot="R270"/>
+<instance part="VCC5" gate="G$1" x="139.7" y="81.28"/>
+<instance part="VCCE1" gate="G$1" x="154.94" y="81.28"/>
+<instance part="VCCE2" gate="G$1" x="177.8" y="68.58"/>
+<instance part="VCCE3" gate="G$1" x="236.22" y="78.74"/>
+<instance part="VCCE4" gate="G$1" x="220.98" y="81.28"/>
+<instance part="C6" gate="G$1" x="226.06" y="73.66"/>
 </instances>
 <busses>
@@
 <pinref part="C16" gate="G$1" pin="P$2"/>
 <pinref part="GND23" gate="G$1" pin="GND"/>
+<pinref part="C6" gate="G$1" pin="P$2"/>
+<wire x1="226.06" y1="71.12" x2="220.98" y2="71.12" width="0.1524" layer="91"/>
+<junction x="220.98" y="71.12"/>
 </segment>
 <segment>
@@
 <wire x1="20.32" y1="152.4" x2="27.94" y2="152.4" width="0.1524" layer="91"/>
 <junction x="27.94" y="152.4"/>
-</segment>
-<segment>
-<pinref part="CN1" gate="G$1" pin="VCC"/>
-<pinref part="VCC18" gate="G$1" pin="VCC"/>
-<wire x1="177.8" y1="66.04" x2="195.58" y2="66.04" width="0.1524" layer="91"/>
-<pinref part="CN1" gate="G$1" pin="SW1"/>
-<wire x1="195.58" y1="66.04" x2="198.12" y2="66.04" width="0.1524" layer="91"/>
-<wire x1="198.12" y1="58.42" x2="195.58" y2="58.42" width="0.1524" layer="91"/>
-<wire x1="195.58" y1="58.42" x2="195.58" y2="66.04" width="0.1524" layer="91"/>
-<junction x="195.58" y="66.04"/>
-</segment>
-<segment>
-<pinref part="C16" gate="G$1" pin="P$1"/>
-<pinref part="VCC19" gate="G$1" pin="VCC"/>
 </segment>
 <segment>
@@
 </segment>
 <segment>
-<pinref part="CN6" gate="A" pin="P$1"/>
-<pinref part="VCC20" gate="G$1" pin="VCC"/>
-<wire x1="236.22" y1="76.2" x2="248.92" y2="76.2" width="0.1524" layer="91"/>
+<pinref part="VCC5" gate="G$1" pin="VCC"/>
+<pinref part="Q2" gate="G$1" pin="S"/>
+<wire x1="139.7" y1="78.74" x2="139.7" y2="76.2" width="0.1524" layer="91"/>
+<wire x1="139.7" y1="76.2" x2="142.24" y2="76.2" width="0.1524" layer="91"/>
 </segment>
 </net>
@@
 <segment>
 <pinref part="C3" gate="G$1" pin="P$1"/>
-<wire x1="20.32" y1="71.12" x2="15.24" y2="71.12" width="0.1524" layer="91"/>
+<wire x1="15.24" y1="73.66" x2="15.24" y2="71.12" width="0.1524" layer="91"/>
 <wire x1="15.24" y1="71.12" x2="10.16" y2="71.12" width="0.1524" layer="91"/>
 <wire x1="10.16" y1="71.12" x2="10.16" y2="68.58" width="0.1524" layer="91"/>
-<wire x1="20.32" y1="71.12" x2="20.32" y2="76.2" width="0.1524" layer="91"/>
-<label x="20.32" y="76.2" size="1.778" layer="95"/>
+<wire x1="15.24" y1="73.66" x2="15.24" y2="76.2" width="0.1524" layer="91"/>
+<label x="15.24" y="76.2" size="1.778" layer="95"/>
 <pinref part="U3" gate="G$1" pin="VIN"/>
 <wire x1="17.78" y1="58.42" x2="15.24" y2="58.42" width="0.1524" layer="91"/>
@@
 <net name="BATSTAT" class="0">
 <segment>
-<pinref part="U1" gate="G$1" pin="PB5"/>
-<wire x1="157.48" y1="106.68" x2="152.4" y2="106.68" width="0.1524" layer="91"/>
-<label x="147.32" y="106.68" size="1.27" layer="95"/>
-</segment>
-<segment>
 <pinref part="U3" gate="G$1" pin="SYSEN"/>
 <wire x1="53.34" y1="40.64" x2="55.88" y2="40.64" width="0.1524" layer="91"/>
@@
 </segment>
 </net>
+<net name="VCCE" class="0">
+<segment>
+<pinref part="VCCE1" gate="G$1" pin="VCCE"/>
+<pinref part="Q2" gate="G$1" pin="D"/>
+<wire x1="154.94" y1="78.74" x2="154.94" y2="76.2" width="0.1524" layer="91"/>
+<wire x1="154.94" y1="76.2" x2="152.4" y2="76.2" width="0.1524" layer="91"/>
+</segment>
+<segment>
+<pinref part="CN1" gate="G$1" pin="VCC"/>
+<wire x1="177.8" y1="66.04" x2="195.58" y2="66.04" width="0.1524" layer="91"/>
+<pinref part="CN1" gate="G$1" pin="SW1"/>
+<wire x1="195.58" y1="66.04" x2="198.12" y2="66.04" width="0.1524" layer="91"/>
+<wire x1="198.12" y1="58.42" x2="195.58" y2="58.42" width="0.1524" layer="91"/>
+<wire x1="195.58" y1="58.42" x2="195.58" y2="66.04" width="0.1524" layer="91"/>
+<junction x="195.58" y="66.04"/>
+<pinref part="VCCE2" gate="G$1" pin="VCCE"/>
+</segment>
+<segment>
+<pinref part="CN6" gate="A" pin="P$1"/>
+<wire x1="236.22" y1="76.2" x2="248.92" y2="76.2" width="0.1524" layer="91"/>
+<pinref part="VCCE3" gate="G$1" pin="VCCE"/>
+</segment>
+<segment>
+<pinref part="C16" gate="G$1" pin="P$1"/>
+<pinref part="VCCE4" gate="G$1" pin="VCCE"/>
+<pinref part="C6" gate="G$1" pin="P$1"/>
+<wire x1="226.06" y1="78.74" x2="220.98" y2="78.74" width="0.1524" layer="91"/>
+<junction x="220.98" y="78.74"/>
+</segment>
+</net>
+<net name="NPWREN" class="0">
+<segment>
+<pinref part="Q2" gate="G$1" pin="G"/>
+<wire x1="144.78" y1="81.28" x2="144.78" y2="86.36" width="0.1524" layer="91"/>
+<wire x1="144.78" y1="86.36" x2="160.02" y2="86.36" width="0.1524" layer="91"/>
+<label x="160.02" y="86.36" size="1.27" layer="95"/>
+</segment>
+<segment>
+<pinref part="U1" gate="G$1" pin="PB5"/>
+<wire x1="157.48" y1="106.68" x2="152.4" y2="106.68" width="0.1524" layer="91"/>
+<label x="147.32" y="106.68" size="1.27" layer="95"/>
+</segment>
+</net>

Commit message: cap on vbat
Parts:
- added C7: 1u, jaw:C0603
Connections:
- net GND: now also C7.P$1
- net N$21: now also C7.P$2
Changed lines of the file:
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@@
 <part name="VCCE4" library="jaw" deviceset="PWR-VCCE" device=""/>
 <part name="C6" library="jaw" deviceset="C" device="0603" value="1u"/>
+<part name="C7" library="jaw" deviceset="C" device="0603" value="1u"/>
 </parts>
 <sheets>
@@
 <instance part="C10" gate="G$1" x="223.52" y="152.4"/>
 <instance part="GND7" gate="G$1" x="223.52" y="144.78"/>
-<instance part="GND8" gate="G$1" x="233.68" y="162.56"/>
+<instance part="GND8" gate="G$1" x="233.68" y="157.48"/>
 <instance part="C11" gate="G$1" x="132.08" y="53.34"/>
 <instance part="R6" gate="G$1" x="50.8" y="177.8"/>
@@
 <instance part="VCCE4" gate="G$1" x="220.98" y="81.28"/>
 <instance part="C6" gate="G$1" x="226.06" y="73.66"/>
+<instance part="C7" gate="G$1" x="226.06" y="165.1" rot="R270"/>
 </instances>
 <busses>
@@
 <segment>
 <pinref part="GND8" gate="G$1" pin="GND"/>
+<wire x1="233.68" y1="160.02" x2="233.68" y2="165.1" width="0.1524" layer="91"/>
+<pinref part="B1" gate="G$1" pin="M"/>
 <wire x1="233.68" y1="165.1" x2="233.68" y2="170.18" width="0.1524" layer="91"/>
-<pinref part="B1" gate="G$1" pin="M"/>
 <wire x1="233.68" y1="170.18" x2="231.14" y2="170.18" width="0.1524" layer="91"/>
+<pinref part="C7" gate="G$1" pin="P$1"/>
+<wire x1="231.14" y1="165.1" x2="233.68" y2="165.1" width="0.1524" layer="91"/>
+<junction x="233.68" y="165.1"/>
 </segment>
 <segment>
@@
 <pinref part="U1" gate="G$1" pin="VBAT"/>
 <wire x1="193.04" y1="162.56" x2="223.52" y2="162.56" width="0.1524" layer="91"/>
-<wire x1="223.52" y1="162.56" x2="223.52" y2="170.18" width="0.1524" layer="91"/>
+<wire x1="223.52" y1="162.56" x2="223.52" y2="165.1" width="0.1524" layer="91"/>
 <pinref part="B1" gate="G$1" pin="P"/>
-</segment>
-</net>
+<pinref part="C7" gate="G$1" pin="P$2"/>
+<wire x1="223.52" y1="165.1" x2="223.52" y2="170.18" width="0.1524" layer="91"/>
+<junction x="223.52" y="165.1"/>
+</segment>
+</net>
