File: cad/epaper.brd (EAGLE design)
At the start: 33.5 x 33.5 mm, 4 parts

Commit message: tweak
Parts:
- added U$2, U$3: FIDUCIAL, adafruit:FIDUCIAL_1MM
- moved C1 4.47 mm to (42.1, 22.1)
- moved SV1 4.47 mm to (36.0, 21.0)
Routing:
- net SPISCK: track 31.6 -> 33.6 mm
- net SPIMOSI: track 27.8 -> 29.8 mm
- net GND: track 37.2 -> 39.2 mm
- net DPYCS: track 27.8 -> 29.8 mm
Other:
- board size 33.5 x 33.5 mm -> 33.5 x 35.5 mm
- board text added: "epaper 128x128"

Commit message: silk text
Parts:
- U$1: value ROBOTMAN-LOGO -> ROBOTMAN-LOGO2; device jaw:ROBOTMAN-LOGO -> jaw:ROBOTMAN-LOGO2
Other:
- board text added: "AMIKETO/epaper"
- board text removed: "mini32/epaper"
Changed lines of the file:
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@@
 <layer number="19" name="Unrouted" color="6" fill="1" visible="yes" active="yes"/>
 <layer number="20" name="Dimension" color="15" fill="1" visible="yes" active="yes"/>
-<layer number="21" name="tPlace" color="7" fill="1" visible="yes" active="yes"/>
+<layer number="21" name="tPlace" color="7" fill="1" visible="no" active="yes"/>
 <layer number="22" name="bPlace" color="7" fill="1" visible="yes" active="yes"/>
 <layer number="23" name="tOrigins" color="15" fill="1" visible="yes" active="yes"/>
@@
 <wire x1="53.3" y1="1" x2="53.8" y2="0.5" width="0" layer="20" curve="90"/>
 <text x="51" y="9" size="2" layer="22" ratio="10" rot="MR0">JAW 2015-03</text>
-<text x="51" y="6" size="1.8" layer="22" ratio="10" rot="MR0">mini32/epaper</text>
+<text x="51" y="6" size="1.6" layer="22" ratio="10" rot="MR0">AMIKETO/epaper</text>
 <text x="31" y="4.5" size="1.5" layer="21" ratio="10">epaper 128x128</text>
 </plain>
@@
 <attribute name="NAME" x="34.77" y="18.3" size="1.27" layer="26" rot="MR90" display="off"/>
 </element>
-<element name="U$1" library="jaw" package="ROBOTMAN-LOGO" value="ROBOTMAN-LOGO" x="57.6" y="11" rot="MR0"/>
+<element name="U$1" library="jaw" package="ROBOTMAN-LOGO2" value="ROBOTMAN-LOGO2" x="57.6" y="11" rot="MR0"/>
 <element name="U$2" library="adafruit" package="FIDUCIAL_1MM" value="FIDUCIAL" x="60" y="33" rot="MR0"/>
 <element name="U$3" library="adafruit" package="FIDUCIAL_1MM" value="FIDUCIAL" x="34" y="13.5" rot="MR0"/>
