File: cad/epaper.brd (EAGLE design)
At the start: 33.5 x 35.5 mm, 6 parts

Commit message: embiggen connector
Parts:
- removed CN1: (no value), jaw:HEADER-2X04
- added CONN2: HEADER-5X2-PTH, jaw:HEADER-5X2-PTH
- C1: value (none) -> .1u
- moved C1 1.06 mm to (42.1, 21.0)
- moved SV1 1.00 mm to (36.0, 20.0)
- moved U$2 1.00 mm to (60.0, 32.0)
- moved U$1 0.10 mm to (57.5, 11.0)
Connections:
- new net N$12: CONN2.9
- new net N$19: CONN2.10
- net DPYCS: now also CONN2.7; no longer CN1.7
- net DPYDC: now also CONN2.6; no longer CN1.6
- net GND: now also CONN2.8; no longer CN1.8
- net NRST: now also CONN2.2; no longer CN1.2
- net SPIMISO: now also CONN2.3; no longer CN1.3
- net SPIMOSI: now also CONN2.5; no longer CN1.5
- net SPISCK: now also CONN2.4; no longer CN1.4
- net VCC: now also CONN2.1; no longer CN1.1
Routing:
- net DPYCS: track 29.8 -> 28.8 mm
- net SPISCK: track 33.6 -> 32.6 mm
- net VCC: track 41.6 -> 42.6 mm
- net SPIMOSI: track 29.8 -> 28.8 mm
- net GND: track 39.2 -> 38.3 mm
Other:
- board size 33.5 x 35.5 mm -> 33.5 x 33.5 mm
- board text added: "JAW 2015-04"
- board text removed: "JAW 2015-03"
