File: cad/oledrgb.brd (EAGLE design)
At the start: 28.5 x 24.5 mm, 13 parts, among them U1 FAN5331SX

Commit message: tweak
Parts:
- added U$1: ROBOTMAN-LOGO, jaw:ROBOTMAN-LOGO
- added U$2, U$3: FIDUCIAL, adafruit:FIDUCIAL_1MM
- C5: value 10u -> .1u
- moved C3 15.2 mm to (42.2, 12.0)
- moved R3 14.9 mm to (59.5, 16.0)
- moved C4 11.5 mm to (44.0, 12.0)
- moved CONN1 9.50 mm to (50.0, 27.0), turned to 180 degrees
- moved C5 2.84 mm to (40.4, 12.0)
- moved C2 0.40 mm to (40.4, 8.50)
- moved R1 0.40 mm to (42.2, 8.50)
- moved R2 0.40 mm to (44.0, 8.50)
- moved CN1 0.20 mm to (58.4, 3.10), turned to 180 degrees
Routing:
- net GND: track 85.8 -> 57.3 mm, vias 2 -> 14
- net SPISCK: track 16.2 -> 32.9 mm, vias 0 -> 2
- net NRST: track 16.6 -> 31.9 mm, vias 0 -> 2
- net V12: track 40.5 -> 52.8 mm
- net SPIMOSI: track 19.5 -> 30.5 mm, vias 0 -> 2
- net VCC: track 45.3 -> 54.8 mm, vias 4 -> 2
- net N$6: track 4.61 -> 14.0 mm
- net N$20: track 4.48 -> 13.4 mm
- net DPYDC: track 20.3 -> 27.3 mm, vias 1 -> 0
- net DPYCS: track 27.6 -> 28.4 mm, vias 1 -> 2
- net N$3: track 6.69 -> 7.21 mm
- added copper zone on layer 1, net GND
Other:
- board size 28.5 x 24.5 mm -> 27.5 x 29.5 mm
- board text added: "RGB 96x64"

Commit message: silk text
Parts:
- added LOGO1: OSHW-LOGOS, Sparkfun-Aesthetics:OSHW-LOGO-S
- U$1: value ROBOTMAN-LOGO -> ROBOTMAN-LOGO2; device jaw:ROBOTMAN-LOGO -> jaw:ROBOTMAN-LOGO2
- moved U$3 17.0 mm to (61.5, 27.5)
- moved U$2 16.1 mm to (37.5, 8.00)
Routing:
- net VCC: track 54.8 -> 52.5 mm
- net GND: track 57.3 -> 55.9 mm, vias 14 -> 16
- net V12: track 52.8 -> 52.2 mm
- net DPYDC: track 27.3 -> 26.8 mm
Other:
- board text added: "JAW 2015-04"
- board text added: "www.amiketo.com"
- board text removed: "JAW 2015-03"
- board text removed: "mini32/RGB OLED"
