File: cad/usb.brd (EAGLE design)
At the start: 21.5 x 14.5 mm, 13 parts, among them CN2 CON_HEADER_1X04, U8 IC_FT230X-SSOP-16

Commit message: silk text
Parts:
- U$1: value ROBOTMAN-LOGO -> ROBOTMAN-LOGO2; device jaw:ROBOTMAN-LOGO -> jaw:ROBOTMAN-LOGO2
Other:
- board text added: "www.amiketo.com"
- board text removed: "www.A791RL.com"
Changed lines of the file:
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@@
 <text x="23" y="7.5" size="2" layer="22" ratio="10" rot="MR0">RX</text>
 <text x="23" y="5" size="2" layer="22" ratio="10" rot="MR0">TX</text>
-<text x="24.5" y="15.3" size="1.25" layer="22" rot="MR0">www.A791RL.com</text>
+<text x="24.5" y="15.3" size="1.25" layer="22" rot="MR0">www.amiketo.com</text>
 </plain>
 <attributes>
@@
 <attribute name="VALUE" x="21.914" y="18.278" size="1" layer="27" font="vector" ratio="10" rot="R270"/>
 </element>
-<element name="U$1" library="jaw" package="ROBOTMAN-LOGO" value="ROBOTMAN-LOGO" x="15" y="9.3" rot="MR0"/>
+<element name="U$1" library="jaw" package="ROBOTMAN-LOGO2" value="ROBOTMAN-LOGO2" x="15" y="9.3" rot="MR0"/>
 <element name="D1" library="jaw" package="SOD-323" value="DIODESOD-323" x="16.8" y="17" smashed="yes" rot="R180">
 <attribute name="NAME" x="15.4" y="18" size="0.75" layer="25" ratio="10"/>
