File: cad/usb.sch (EAGLE design)
At the start: 13 parts, among them CN2 CON_HEADER_1X04, U8 IC_FT230X-SSOP-16

Commit message: silk text
Parts:
- U$1: value ROBOTMAN-LOGO -> ROBOTMAN-LOGO2; device jaw:ROBOTMAN-LOGO -> jaw:ROBOTMAN-LOGO2
Changed lines of the file:
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@@
 <part name="C3" library="jaw" deviceset="C" device="0603" value="1+u"/>
 <part name="GND5" library="jaw" deviceset="PWR-GND" device=""/>
-<part name="U$1" library="jaw" deviceset="ROBOTMAN-LOGO" device=""/>
+<part name="U$1" library="jaw" deviceset="ROBOTMAN-LOGO" device="2" value="ROBOTMAN-LOGO2"/>
 <part name="D1" library="jaw" deviceset="DIODE" device="SOD-323"/>
 </parts>
