File: cad/amiketo.sch (EAGLE design)
At the start: 56 parts, among them CN1 MICROSD-EJECT, J1 HEADER-5X1, Q1 IRLML6344TRPBF, Q2 DMP2035U-7, SW2 SWITCHKMR211, SW3 SWITCHKMR211, U1 STM32F411/48, U2 LIS3DH, U3 ADP5062, U4 MCP1824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

Commit message: tweak
Parts:
- added D2: 1A, jaw:DIODE-0805
- D1: value DIODESOD-323 -> 200mA
- F1: value FUSE -> 750mA
Connections:
- removed net VUSB: C3.P$1, F1.2, JP1.12, U3.VIN
- new net N$24: D2.A, F1.2
- new net VIN: C3.P$1, D2.C, JP1.12, U3.VIN
Other:
- moved on the sheet: C14, R6, R7
Changed lines of the file:
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@@
 <part name="U1" library="jaw" deviceset="STM32F411/48" device=""/>
 <part name="U4" library="jaw" deviceset="MCP1824" device=""/>
-<part name="USB1" library="dp_devices" deviceset="CON-USB-F" device="-MICRO-B"/>
+<part name="USB1" library="dp_devices" deviceset="CON-USB-F" device="-MICRO-B" value=""/>
 <part name="CN3" library="adafruit" deviceset="JST_2PIN" device="-SMT-RA"/>
-<part name="F1" library="jaw" deviceset="FUSE" device=""/>
+<part name="F1" library="jaw" deviceset="FUSE" device="" value="750mA"/>
 <part name="C1" library="jaw" deviceset="C" device="0603" value="10u"/>
 <part name="C2" library="jaw" deviceset="C" device="0603" value="1u"/>
@@
 <part name="C4" library="jaw" deviceset="C" device="0603" value="4u7"/>
 <part name="GND1" library="jaw" deviceset="PWR-GND" device=""/>
-<part name="GND2" library="jaw" deviceset="PWR-GND" device=""/>
 <part name="GND3" library="jaw" deviceset="PWR-GND" device=""/>
 <part name="SW2" library="jaw" deviceset="SWITCH" device="KMR211"/>
@@
 <part name="GND9" library="jaw" deviceset="PWR-GND" device=""/>
 <part name="SPKR1" library="jaw" deviceset="PUI-5040" device=""/>
-<part name="D1" library="jaw" deviceset="DIODE" device="SOD-323"/>
+<part name="D1" library="jaw" deviceset="DIODE" device="SOD-323" value="200mA"/>
 <part name="VCC3" library="jaw" deviceset="PWR-VCC" device=""/>
 <part name="GND10" library="jaw" deviceset="PWR-GND" device=""/>
@@
 <part name="GND4" library="jaw" deviceset="PWR-GND" device=""/>
 <part name="VCC6" library="jaw" deviceset="PWR-VCC" device=""/>
+<part name="D2" library="jaw" deviceset="DIODE" device="-0805" value="1A"/>
 </parts>
 <sheets>
@@
 <instance part="C4" gate="G$1" x="86.36" y="25.4"/>
 <instance part="GND1" gate="G$1" x="43.18" y="10.16"/>
-<instance part="GND2" gate="G$1" x="73.66" y="182.88"/>
 <instance part="GND3" gate="G$1" x="109.22" y="40.64"/>
 <instance part="SW2" gate="G$1" x="104.14" y="193.04"/>
@@
 <instance part="GND8" gate="G$1" x="233.68" y="157.48"/>
 <instance part="C11" gate="G$1" x="132.08" y="53.34"/>
-<instance part="R6" gate="G$1" x="50.8" y="177.8"/>
-<instance part="R7" gate="G$1" x="50.8" y="170.18"/>
+<instance part="R6" gate="G$1" x="48.26" y="172.72"/>
+<instance part="R7" gate="G$1" x="48.26" y="165.1"/>
 <instance part="LED1" gate="G$1" x="43.18" y="127" rot="R270"/>
 <instance part="R8" gate="G$1" x="43.18" y="139.7" rot="R270"/>
@@
 <instance part="U$2" gate="G$1" x="271.78" y="25.4"/>
 <instance part="U$3" gate="G$1" x="271.78" y="33.02"/>
-<instance part="C14" gate="G$1" x="132.08" y="119.38"/>
+<instance part="C14" gate="G$1" x="116.84" y="121.92"/>
 <instance part="GND12" gate="G$1" x="99.06" y="81.28"/>
-<instance part="GND14" gate="G$1" x="132.08" y="86.36"/>
+<instance part="GND14" gate="G$1" x="116.84" y="116.84"/>
 <instance part="VCC4" gate="G$1" x="99.06" y="132.08"/>
 <instance part="GND19" gate="G$1" x="30.48" y="167.64"/>
@@
 <instance part="VCCE1" gate="G$1" x="154.94" y="81.28"/>
 <instance part="VCCE2" gate="G$1" x="177.8" y="68.58"/>
-<instance part="VCCE3" gate="G$1" x="236.22" y="78.74"/>
+<instance part="VCCE3" gate="G$1" x="236.22" y="81.28"/>
 <instance part="VCCE4" gate="G$1" x="220.98" y="81.28"/>
 <instance part="C6" gate="G$1" x="226.06" y="73.66"/>
@@
 <instance part="GND4" gate="G$1" x="193.04" y="187.96"/>
 <instance part="VCC6" gate="G$1" x="193.04" y="200.66"/>
+<instance part="D2" gate="G$1" x="58.42" y="182.88"/>
 </instances>
 <busses>
@@
 <pinref part="GND26" gate="G$1" pin="GND"/>
 <pinref part="C23" gate="G$1" pin="P$2"/>
-</segment>
-<segment>
-<pinref part="USB1" gate="USB" pin="GND"/>
-<wire x1="30.48" y1="185.42" x2="73.66" y2="185.42" width="0.1524" layer="91"/>
-<pinref part="GND2" gate="G$1" pin="GND"/>
 </segment>
 <segment>
@@
 </segment>
 <segment>
-<wire x1="132.08" y1="109.22" x2="132.08" y2="96.52" width="0.1524" layer="91"/>
 <pinref part="GND14" gate="G$1" pin="GND"/>
-<wire x1="132.08" y1="96.52" x2="132.08" y2="88.9" width="0.1524" layer="91"/>
-<wire x1="132.08" y1="114.3" x2="132.08" y2="109.22" width="0.1524" layer="91"/>
 <pinref part="C14" gate="G$1" pin="P$2"/>
-<wire x1="132.08" y1="116.84" x2="132.08" y2="114.3" width="0.1524" layer="91"/>
 </segment>
 <segment>
 <pinref part="USB1" gate="USB" pin="USBID"/>
 <pinref part="GND19" gate="G$1" pin="GND"/>
-<wire x1="30.48" y1="170.18" x2="30.48" y2="175.26" width="0.1524" layer="91"/>
+<wire x1="30.48" y1="170.18" x2="30.48" y2="172.72" width="0.1524" layer="91"/>
+<wire x1="30.48" y1="172.72" x2="30.48" y2="175.26" width="0.1524" layer="91"/>
+<wire x1="30.48" y1="172.72" x2="35.56" y2="172.72" width="0.1524" layer="91"/>
+<junction x="30.48" y="172.72"/>
+<pinref part="USB1" gate="USB" pin="GND"/>
+<wire x1="30.48" y1="185.42" x2="35.56" y2="185.42" width="0.1524" layer="91"/>
+<wire x1="35.56" y1="172.72" x2="35.56" y2="185.42" width="0.1524" layer="91"/>
 </segment>
 <segment>
@@
 <segment>
 <pinref part="C14" gate="G$1" pin="P$1"/>
-<wire x1="132.08" y1="124.46" x2="132.08" y2="127" width="0.1524" layer="91"/>
-<wire x1="132.08" y1="127" x2="101.6" y2="127" width="0.1524" layer="91"/>
+<wire x1="116.84" y1="127" x2="101.6" y2="127" width="0.1524" layer="91"/>
 <wire x1="101.6" y1="127" x2="101.6" y2="124.46" width="0.1524" layer="91"/>
 <wire x1="101.6" y1="127" x2="99.06" y2="127" width="0.1524" layer="91"/>
@@
 </segment>
 </net>
-<net name="VUSB" class="0">
-<segment>
-<pinref part="F1" gate="G$1" pin="2"/>
-<wire x1="55.88" y1="182.88" x2="63.5" y2="182.88" width="0.1524" layer="91"/>
-<label x="63.5" y="182.88" size="1.27" layer="95"/>
-</segment>
+<net name="VIN" class="0">
 <segment>
 <pinref part="C3" gate="G$1" pin="P$1"/>
@@
 <wire x1="254" y1="116.84" x2="246.38" y2="116.84" width="0.1524" layer="91"/>
 <label x="238.76" y="116.84" size="1.27" layer="95"/>
+</segment>
+<segment>
+<pinref part="D2" gate="G$1" pin="C"/>
+<wire x1="60.96" y1="182.88" x2="63.5" y2="182.88" width="0.1524" layer="91"/>
+<label x="63.5" y="182.88" size="1.27" layer="95"/>
 </segment>
 </net>
@@
 <pinref part="USB1" gate="USB" pin="D-"/>
 <pinref part="R6" gate="G$1" pin="P$1"/>
-<wire x1="30.48" y1="180.34" x2="45.72" y2="180.34" width="0.1524" layer="91"/>
-<wire x1="45.72" y1="180.34" x2="45.72" y2="177.8" width="0.1524" layer="91"/>
+<wire x1="30.48" y1="180.34" x2="40.64" y2="180.34" width="0.1524" layer="91"/>
+<wire x1="40.64" y1="180.34" x2="40.64" y2="172.72" width="0.1524" layer="91"/>
+<wire x1="40.64" y1="172.72" x2="43.18" y2="172.72" width="0.1524" layer="91"/>
 </segment>
 </net>
@@
 <segment>
 <pinref part="USB1" gate="USB" pin="D+"/>
-<wire x1="30.48" y1="177.8" x2="43.18" y2="177.8" width="0.1524" layer="91"/>
-<wire x1="43.18" y1="177.8" x2="43.18" y2="170.18" width="0.1524" layer="91"/>
+<wire x1="30.48" y1="177.8" x2="38.1" y2="177.8" width="0.1524" layer="91"/>
+<wire x1="38.1" y1="177.8" x2="38.1" y2="165.1" width="0.1524" layer="91"/>
 <pinref part="R7" gate="G$1" pin="P$1"/>
-<wire x1="43.18" y1="170.18" x2="45.72" y2="170.18" width="0.1524" layer="91"/>
+<wire x1="38.1" y1="165.1" x2="43.18" y2="165.1" width="0.1524" layer="91"/>
 </segment>
 </net>
@@
 <segment>
 <pinref part="R6" gate="G$1" pin="P$2"/>
-<wire x1="55.88" y1="177.8" x2="63.5" y2="177.8" width="0.1524" layer="91"/>
-<label x="63.5" y="177.8" size="1.27" layer="95"/>
+<wire x1="53.34" y1="172.72" x2="63.5" y2="172.72" width="0.1524" layer="91"/>
+<label x="63.5" y="172.72" size="1.27" layer="95"/>
 </segment>
 <segment>
@@
 <segment>
 <pinref part="R7" gate="G$1" pin="P$2"/>
-<wire x1="55.88" y1="170.18" x2="63.5" y2="170.18" width="0.1524" layer="91"/>
-<label x="63.5" y="170.18" size="1.27" layer="95"/>
+<wire x1="53.34" y1="165.1" x2="63.5" y2="165.1" width="0.1524" layer="91"/>
+<label x="63.5" y="165.1" size="1.27" layer="95"/>
 </segment>
 <segment>
@@
 <segment>
 <pinref part="CN6" gate="A" pin="P$1"/>
-<wire x1="236.22" y1="76.2" x2="248.92" y2="76.2" width="0.1524" layer="91"/>
+<wire x1="236.22" y1="78.74" x2="236.22" y2="76.2" width="0.1524" layer="91"/>
+<wire x1="236.22" y1="76.2" x2="238.76" y2="76.2" width="0.1524" layer="91"/>
+<wire x1="238.76" y1="76.2" x2="248.92" y2="76.2" width="0.1524" layer="91"/>
 <pinref part="VCCE3" gate="G$1" pin="VCCE"/>
 </segment>
@@
 </segment>
 </net>
+<net name="N$24" class="0">
+<segment>
+<pinref part="F1" gate="G$1" pin="2"/>
+<pinref part="D2" gate="G$1" pin="A"/>
+</segment>
+</net>

Commit message: i2c r, tweak
Parts:
- added R3, R9: 10k, jaw:R0603
Connections:
- net I2CCL: now also R3.P$1
- net I2CDA: now also R9.P$1
- net VCC: now also R3.P$2, R9.P$2
Changed lines of the file:
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@@
 <setting verticaltext="up"/>
 </settings>
-<grid distance="0.1" unitdist="inch" unit="inch" style="lines" multiple="1" display="yes" altdistance="0.01" altunitdist="inch" altunit="inch"/>
+<grid distance="0.1" unitdist="inch" unit="inch" style="lines" multiple="1" display="no" altdistance="0.01" altunitdist="inch" altunit="inch"/>
 <layers>
 <layer number="1" name="Top" color="4" fill="1" visible="no" active="no"/>
@@
 <part name="VCC6" library="jaw" deviceset="PWR-VCC" device=""/>
 <part name="D2" library="jaw" deviceset="DIODE" device="-0805" value="1A"/>
+<part name="R3" library="jaw" deviceset="R" device="0603" value="10k"/>
+<part name="R9" library="jaw" deviceset="R" device="0603" value="10k"/>
+<part name="VCC7" library="jaw" deviceset="PWR-VCC" device=""/>
 </parts>
 <sheets>
@@
 <instance part="VCC6" gate="G$1" x="193.04" y="200.66"/>
 <instance part="D2" gate="G$1" x="58.42" y="182.88"/>
+<instance part="R3" gate="G$1" x="137.16" y="114.3" rot="R90"/>
+<instance part="R9" gate="G$1" x="142.24" y="114.3" rot="R90"/>
+<instance part="VCC7" gate="G$1" x="139.7" y="124.46"/>
 </instances>
 <busses>
@@
 <pinref part="VCC6" gate="G$1" pin="VCC"/>
 </segment>
+<segment>
+<pinref part="R3" gate="G$1" pin="P$2"/>
+<pinref part="R9" gate="G$1" pin="P$2"/>
+<wire x1="137.16" y1="119.38" x2="139.7" y2="119.38" width="0.1524" layer="91"/>
+<pinref part="VCC7" gate="G$1" pin="VCC"/>
+<wire x1="139.7" y1="119.38" x2="142.24" y2="119.38" width="0.1524" layer="91"/>
+<wire x1="139.7" y1="119.38" x2="139.7" y2="121.92" width="0.1524" layer="91"/>
+<junction x="139.7" y="119.38"/>
+</segment>
 </net>
 <net name="BOOT0" class="0">
@@
 <segment>
 <pinref part="U1" gate="G$1" pin="PB6"/>
-<wire x1="157.48" y1="104.14" x2="152.4" y2="104.14" width="0.1524" layer="91"/>
-<label x="147.32" y="104.14" size="1.27" layer="95"/>
+<wire x1="157.48" y1="104.14" x2="137.16" y2="104.14" width="0.1524" layer="91"/>
+<label x="127" y="104.14" size="1.27" layer="95"/>
+<pinref part="R3" gate="G$1" pin="P$1"/>
+<wire x1="137.16" y1="104.14" x2="132.08" y2="104.14" width="0.1524" layer="91"/>
+<wire x1="137.16" y1="109.22" x2="137.16" y2="104.14" width="0.1524" layer="91"/>
+<junction x="137.16" y="104.14"/>
 </segment>
 <segment>
@@
 <segment>
 <pinref part="U1" gate="G$1" pin="PB7"/>
-<wire x1="157.48" y1="101.6" x2="152.4" y2="101.6" width="0.1524" layer="91"/>
-<label x="147.32" y="101.6" size="1.27" layer="95"/>
-</segment>
-<segment>
+<wire x1="157.48" y1="101.6" x2="142.24" y2="101.6" width="0.1524" layer="91"/>
+<label x="127" y="101.6" size="1.27" layer="95"/>
+<pinref part="R9" gate="G$1" pin="P$1"/>
+<wire x1="142.24" y1="101.6" x2="132.08" y2="101.6" width="0.1524" layer="91"/>
+<wire x1="142.24" y1="109.22" x2="142.24" y2="101.6" width="0.1524" layer="91"/>
+<junction x="142.24" y="101.6"/>
+</segment>
+<segment>

Commit message: swap regulator
Parts:
- removed CN6: (no value), jaw:HEADER-2X4
- removed U4: MCP1824, jaw:MCP1824
- added CONN1: HEADER-5X2-PTH, jaw:HEADER-5X2-PTH
- added R10, R11: 1M, jaw:R0603
- added VR1: mcp1700 /3v3, jaw:REGULATOR-SOT23-3
Connections:
- net DPYCS: now also CONN1.7; no longer CN6.P$7
- net DPYDC: now also CONN1.6; no longer CN6.P$6
- net GND: now also CONN1.8, R10.P$2, VR1.GND; no longer CN6.P$8, U4.GND
- net I2CCL: now also CONN1.9
- net I2CDA: now also CONN1.10
- net N$9: now also R10.P$1
- net NPWREN: now also R11.P$2
- net NRST: now also CONN1.2; no longer CN6.P$2
- net SPIMISO: now also CONN1.3; no longer CN6.P$3
- net SPIMOSI: now also CONN1.5; no longer CN6.P$5
- net SPISCK: now also CONN1.4; no longer CN6.P$4
- net VCC: now also R11.P$1, VR1.VO; no longer U4.VOUT
- net VCCE: now also CONN1.1; no longer CN6.P$1
- net VP: now also VR1.VI; no longer U4.NSHTDN, U4.VIN
Other:
- moved on the sheet: Q2, R2
