File: cad/amiketo.sch (EAGLE design)
At the start: 61 parts, among them CN1 MICROSD-EJECT, J1 HEADER-5X1, Q1 IRLML6344TRPBF, Q2 DMP2035U-7, SW2 SWITCHKMR211, SW3 SWITCHKMR211, U1 STM32F411/48, U2 LIS3DH, U3 ADP5062, U5 MAX17048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

Commit message: tweak
Other:
- moved on the sheet: C1, C11, C12, C14, C16, C17, C2, C3, C4, C5, C6, CN1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

Commit message: display reset
Parts:
- added C13: .001u, jaw:C0603
- added D3: any, jaw:DIODESOD-323
- added R12: 4k7, jaw:R0603
Connections:
- new net NRST2: C13.P$1, CONN1.2, D3.A, R12.P$1
- net GND: now also C13.P$2
- net NRST: now also D3.C; no longer CONN1.2
- net VCCE: now also R12.P$2
Other:
- note added: "generate reset for display after Q2 is turned on"
- moved on the sheet: Q2, R11
Changed lines of the file:
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@@
 <setting verticaltext="up"/>
 </settings>
-<grid distance="0.1" unitdist="inch" unit="inch" style="lines" multiple="1" display="yes" altdistance="0.01" altunitdist="inch" altunit="inch"/>
+<grid distance="0.1" unitdist="inch" unit="inch" style="lines" multiple="1" display="no" altdistance="0.01" altunitdist="inch" altunit="inch"/>
 <layers>
 <layer number="1" name="Top" color="4" fill="1" visible="no" active="no"/>
@@
 <part name="VR1" library="jaw" deviceset="REGULATOR" device="-SOT23-3" value="mcp1700 /3v3"/>
 <part name="FRAME2" library="frames" deviceset="FRAME_B_L" device=""/>
+<part name="R12" library="jaw" deviceset="R" device="0603" value="4k7"/>
+<part name="C13" library="jaw" deviceset="C" device="0603" value=".001u"/>
+<part name="GND2" library="jaw" deviceset="PWR-GND" device=""/>
+<part name="D3" library="jaw" deviceset="DIODE" device="SOD-323" value="any"/>
 </parts>
 <sheets>
@@
 <text x="381" y="73.66" size="3.81" layer="97">display</text>
 <text x="373.38" y="114.3" size="3.81" layer="97">JTAG/SWD</text>
-<text x="223.52" y="68.58" size="1.27" layer="97">to reduce leakage current
+<text x="226.06" y="63.5" size="1.27" layer="97">to reduce leakage current
 thru dpy + sd card while off</text>
+<text x="210.82" y="43.18" size="1.27" layer="97">generate reset for display
+after Q2 is turned on</text>
 </plain>
 <instances>
@@
 <instance part="U$1" gate="G$1" x="388.62" y="25.4"/>
 <instance part="R2" gate="G$1" x="299.72" y="193.04"/>
-<instance part="Q2" gate="G$1" x="215.9" y="55.88" rot="R180"/>
-<instance part="VCC5" gate="G$1" x="215.9" y="71.12"/>
+<instance part="Q2" gate="G$1" x="223.52" y="55.88" rot="MR180"/>
+<instance part="VCC5" gate="G$1" x="223.52" y="73.66"/>
 <instance part="VCCE1" gate="G$1" x="241.3" y="55.88"/>
 <instance part="VCCE2" gate="G$1" x="287.02" y="60.96"/>
@@
 <instance part="CONN1" gate="G$1" x="386.08" y="55.88"/>
 <instance part="R10" gate="G$1" x="304.8" y="187.96" rot="R270"/>
-<instance part="R11" gate="G$1" x="223.52" y="63.5"/>
+<instance part="R11" gate="G$1" x="215.9" y="63.5" rot="R180"/>
 <instance part="VR1" gate="G$1" x="119.38" y="66.04" smashed="yes">
 <attribute name="NAME" x="109.22" y="58.42" size="2.54" layer="95" ratio="10"/>
@@
 <instance part="FRAME2" gate="G$1" x="0" y="0"/>
 <instance part="FRAME2" gate="G$2" x="325.12" y="0"/>
+<instance part="R12" gate="G$1" x="241.3" y="40.64" rot="R90"/>
+<instance part="C13" gate="G$1" x="241.3" y="30.48"/>
+<instance part="GND2" gate="G$1" x="241.3" y="25.4"/>
+<instance part="D3" gate="G$1" x="233.68" y="35.56" rot="R180"/>
 </instances>
 <busses>
@@
 <label x="396.24" y="58.42" size="1.778" layer="95"/>
 </segment>
+<segment>
+<pinref part="C13" gate="G$1" pin="P$2"/>
+<pinref part="GND2" gate="G$1" pin="GND"/>
+</segment>
 </net>
 <net name="VCC" class="0">
@@
 <pinref part="VCC5" gate="G$1" pin="VCC"/>
 <pinref part="Q2" gate="G$1" pin="S"/>
-<wire x1="215.9" y1="68.58" x2="215.9" y2="63.5" width="0.1524" layer="91"/>
-<wire x1="215.9" y1="63.5" x2="215.9" y2="60.96" width="0.1524" layer="91"/>
+<wire x1="223.52" y1="71.12" x2="223.52" y2="63.5" width="0.1524" layer="91"/>
+<wire x1="223.52" y1="63.5" x2="223.52" y2="60.96" width="0.1524" layer="91"/>
 <pinref part="R11" gate="G$1" pin="P$1"/>
-<wire x1="218.44" y1="63.5" x2="215.9" y2="63.5" width="0.1524" layer="91"/>
-<junction x="215.9" y="63.5"/>
+<wire x1="220.98" y1="63.5" x2="223.52" y2="63.5" width="0.1524" layer="91"/>
+<junction x="223.52" y="63.5"/>
 </segment>
 <segment>
@@
 <pinref part="U1" gate="G$1" pin="BOOT0"/>
 <wire x1="149.86" y1="165.1" x2="157.48" y2="165.1" width="0.1524" layer="91"/>
+<label x="134.62" y="172.72" size="1.778" layer="95"/>
 </segment>
 <segment>
@@
 <pinref part="U1" gate="G$1" pin="NRST"/>
 <wire x1="152.4" y1="167.64" x2="157.48" y2="167.64" width="0.1524" layer="91"/>
+<label x="134.62" y="193.04" size="1.778" layer="95"/>
 </segment>
 <segment>
@@
 </segment>
 <segment>
-<pinref part="CONN1" gate="G$1" pin="2"/>
-<wire x1="393.7" y1="66.04" x2="396.24" y2="66.04" width="0.1524" layer="91"/>
-<label x="396.24" y="66.04" size="1.778" layer="95"/>
+<pinref part="D3" gate="G$1" pin="C"/>
+<wire x1="231.14" y1="35.56" x2="226.06" y2="35.56" width="0.1524" layer="91"/>
+<label x="220.98" y="35.56" size="1.778" layer="95"/>
 </segment>
 </net>
@@
 <pinref part="Q2" gate="G$1" pin="D"/>
 <wire x1="241.3" y1="53.34" x2="241.3" y2="50.8" width="0.1524" layer="91"/>
-<wire x1="241.3" y1="50.8" x2="215.9" y2="50.8" width="0.1524" layer="91"/>
+<wire x1="241.3" y1="50.8" x2="223.52" y2="50.8" width="0.1524" layer="91"/>
+<pinref part="R12" gate="G$1" pin="P$2"/>
+<wire x1="241.3" y1="45.72" x2="241.3" y2="50.8" width="0.1524" layer="91"/>
+<junction x="241.3" y="50.8"/>
 </segment>
 <segment>
@@
 <segment>
 <pinref part="Q2" gate="G$1" pin="G"/>
-<wire x1="220.98" y1="58.42" x2="228.6" y2="58.42" width="0.1524" layer="91"/>
-<wire x1="228.6" y1="58.42" x2="228.6" y2="63.5" width="0.1524" layer="91"/>
-<wire x1="228.6" y1="63.5" x2="246.38" y2="63.5" width="0.1524" layer="91"/>
-<label x="246.38" y="63.5" size="1.27" layer="95"/>
+<wire x1="218.44" y1="58.42" x2="210.82" y2="58.42" width="0.1524" layer="91"/>
+<wire x1="210.82" y1="58.42" x2="210.82" y2="63.5" width="0.1524" layer="91"/>
+<wire x1="210.82" y1="63.5" x2="205.74" y2="63.5" width="0.1524" layer="91"/>
+<label x="200.66" y="63.5" size="1.27" layer="95"/>
 <pinref part="R11" gate="G$1" pin="P$2"/>
-<junction x="228.6" y="63.5"/>
+<junction x="210.82" y="63.5"/>
 </segment>
 <segment>
@@
 </segment>
 </net>
+<net name="NRST2" class="0">
+<segment>
+<pinref part="R12" gate="G$1" pin="P$1"/>
+<pinref part="C13" gate="G$1" pin="P$1"/>
+<pinref part="D3" gate="G$1" pin="A"/>
+<wire x1="236.22" y1="35.56" x2="241.3" y2="35.56" width="0.1524" layer="91"/>
+<junction x="241.3" y="35.56"/>
+<wire x1="241.3" y1="35.56" x2="248.92" y2="35.56" width="0.1524" layer="91"/>
+<label x="248.92" y="35.56" size="1.778" layer="95"/>
+</segment>
+<segment>
+<pinref part="CONN1" gate="G$1" pin="2"/>
+<wire x1="393.7" y1="66.04" x2="396.24" y2="66.04" width="0.1524" layer="91"/>
+<label x="396.24" y="66.04" size="1.778" layer="95"/>
+</segment>
+</net>

Commit message: tweak
Parts:
- D1: value 200mA -> any
Changed lines of the file:
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@@
 <part name="GND9" library="jaw" deviceset="PWR-GND" device=""/>
 <part name="SPKR1" library="jaw" deviceset="PUI-5040" device=""/>
-<part name="D1" library="jaw" deviceset="DIODE" device="SOD-323" value="200mA"/>
+<part name="D1" library="jaw" deviceset="DIODE" device="SOD-323" value="any"/>
 <part name="VCC3" library="jaw" deviceset="PWR-VCC" device=""/>
 <part name="GND10" library="jaw" deviceset="PWR-GND" device=""/>

Commit message: tweak silk
Parts:
- C8, C9: value 5p -> 4p7
Changed lines of the file:
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@@
 <part name="C5" library="jaw" deviceset="C" device="0603" value="10u"/>
 <part name="X2" library="jaw" deviceset="XTAL" device="32X15" value="32k768"/>
-<part name="C8" library="jaw" deviceset="C" device="0603" value="5p"/>
-<part name="C9" library="jaw" deviceset="C" device="0603" value="5p"/>
+<part name="C8" library="jaw" deviceset="C" device="0603" value="4p7"/>
+<part name="C9" library="jaw" deviceset="C" device="0603" value="4p7"/>
 <part name="GND5" library="jaw" deviceset="PWR-GND" device=""/>
 <part name="GND6" library="jaw" deviceset="PWR-GND" device=""/>

Commit message: add info
Other:
- note added: "configure gpio with pullup"
- moved on the sheet: C12, R3, R9
Changed lines of the file:
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@@
 <setting verticaltext="up"/>
 </settings>
-<grid distance="0.1" unitdist="inch" unit="inch" style="lines" multiple="1" display="no" altdistance="0.01" altunitdist="inch" altunit="inch"/>
+<grid distance="0.1" unitdist="inch" unit="inch" style="lines" multiple="1" display="yes" altdistance="0.01" altunitdist="inch" altunit="inch"/>
 <layers>
 <layer number="1" name="Top" color="4" fill="1" visible="no" active="no"/>
@@
 <text x="210.82" y="43.18" size="1.27" layer="97">generate reset for display
 after Q2 is turned on</text>
+<wire x1="355.6" y1="38.1" x2="355.6" y2="86.36" width="0.635" layer="97"/>
+<wire x1="355.6" y1="86.36" x2="424.18" y2="86.36" width="0.635" layer="97"/>
+<wire x1="355.6" y1="88.9" x2="355.6" y2="134.62" width="0.635" layer="97"/>
+<wire x1="355.6" y1="134.62" x2="424.18" y2="134.62" width="0.635" layer="97"/>
+<wire x1="355.6" y1="137.16" x2="355.6" y2="218.44" width="0.635" layer="97"/>
+<wire x1="266.7" y1="228.6" x2="266.7" y2="172.72" width="0.635" layer="97"/>
+<wire x1="266.7" y1="172.72" x2="353.06" y2="172.72" width="0.635" layer="97"/>
+<wire x1="266.7" y1="170.18" x2="266.7" y2="96.52" width="0.635" layer="97"/>
+<wire x1="266.7" y1="96.52" x2="353.06" y2="96.52" width="0.635" layer="97"/>
+<wire x1="266.7" y1="91.44" x2="266.7" y2="5.08" width="0.635" layer="97"/>
+<wire x1="7.62" y1="91.44" x2="195.58" y2="91.44" width="0.635" layer="97"/>
+<wire x1="195.58" y1="91.44" x2="195.58" y2="5.08" width="0.635" layer="97"/>
+<wire x1="198.12" y1="91.44" x2="266.7" y2="91.44" width="0.635" layer="97"/>
+<wire x1="86.36" y1="93.98" x2="86.36" y2="154.94" width="0.635" layer="97"/>
+<text x="294.64" y="48.26" size="1.27" layer="97" ratio="10">configure gpio with pullup</text>
 </plain>
 <instances>
@@
 <instance part="U2" gate="G$1" x="314.96" y="134.62"/>
 <instance part="JP1" gate="G$1" x="391.16" y="175.26"/>
-<instance part="C12" gate="G$1" x="355.6" y="104.14"/>
-<instance part="GND4" gate="G$1" x="355.6" y="99.06"/>
-<instance part="VCC6" gate="G$1" x="355.6" y="111.76"/>
+<instance part="C12" gate="G$1" x="414.02" y="104.14"/>
+<instance part="GND4" gate="G$1" x="414.02" y="99.06"/>
+<instance part="VCC6" gate="G$1" x="414.02" y="111.76"/>
 <instance part="D2" gate="G$1" x="63.5" y="137.16"/>
-<instance part="R3" gate="G$1" x="137.16" y="114.3" rot="R90"/>
-<instance part="R9" gate="G$1" x="142.24" y="114.3" rot="R90"/>
-<instance part="VCC7" gate="G$1" x="139.7" y="124.46"/>
+<instance part="R3" gate="G$1" x="132.08" y="114.3" rot="R90"/>
+<instance part="R9" gate="G$1" x="139.7" y="114.3" rot="R90"/>
+<instance part="VCC7" gate="G$1" x="134.62" y="124.46"/>
 <instance part="CONN1" gate="G$1" x="386.08" y="55.88"/>
 <instance part="R10" gate="G$1" x="304.8" y="187.96" rot="R270"/>
@@
 <pinref part="R3" gate="G$1" pin="P$2"/>
 <pinref part="R9" gate="G$1" pin="P$2"/>
-<wire x1="137.16" y1="119.38" x2="139.7" y2="119.38" width="0.1524" layer="91"/>
+<wire x1="132.08" y1="119.38" x2="134.62" y2="119.38" width="0.1524" layer="91"/>
 <pinref part="VCC7" gate="G$1" pin="VCC"/>
-<wire x1="139.7" y1="119.38" x2="142.24" y2="119.38" width="0.1524" layer="91"/>
-<wire x1="139.7" y1="119.38" x2="139.7" y2="121.92" width="0.1524" layer="91"/>
-<junction x="139.7" y="119.38"/>
+<wire x1="134.62" y1="119.38" x2="139.7" y2="119.38" width="0.1524" layer="91"/>
+<wire x1="134.62" y1="119.38" x2="134.62" y2="121.92" width="0.1524" layer="91"/>
+<junction x="134.62" y="119.38"/>
 </segment>
 </net>
@@
 <pinref part="CN1" gate="G$1" pin="SW1"/>
 <wire x1="307.34" y1="50.8" x2="304.8" y2="50.8" width="0.1524" layer="91"/>
-<label x="297.18" y="50.8" size="1.27" layer="95"/>
+<label x="294.64" y="50.8" size="1.778" layer="95"/>
 </segment>
 </net>
@@
 <segment>
 <pinref part="U1" gate="G$1" pin="PB6"/>
-<wire x1="157.48" y1="104.14" x2="137.16" y2="104.14" width="0.1524" layer="91"/>
-<label x="127" y="104.14" size="1.27" layer="95"/>
+<wire x1="157.48" y1="104.14" x2="132.08" y2="104.14" width="0.1524" layer="91"/>
+<label x="121.92" y="104.14" size="1.27" layer="95"/>
 <pinref part="R3" gate="G$1" pin="P$1"/>
-<wire x1="137.16" y1="104.14" x2="132.08" y2="104.14" width="0.1524" layer="91"/>
-<wire x1="137.16" y1="109.22" x2="137.16" y2="104.14" width="0.1524" layer="91"/>
-<junction x="137.16" y="104.14"/>
+<wire x1="132.08" y1="104.14" x2="127" y2="104.14" width="0.1524" layer="91"/>
+<wire x1="132.08" y1="109.22" x2="132.08" y2="104.14" width="0.1524" layer="91"/>
+<junction x="132.08" y="104.14"/>
 </segment>
 <segment>
@@
 <segment>
 <pinref part="U1" gate="G$1" pin="PB7"/>
-<wire x1="157.48" y1="101.6" x2="142.24" y2="101.6" width="0.1524" layer="91"/>
-<label x="127" y="101.6" size="1.27" layer="95"/>
+<wire x1="157.48" y1="101.6" x2="139.7" y2="101.6" width="0.1524" layer="91"/>
+<label x="121.92" y="101.6" size="1.27" layer="95"/>
 <pinref part="R9" gate="G$1" pin="P$1"/>
-<wire x1="142.24" y1="101.6" x2="132.08" y2="101.6" width="0.1524" layer="91"/>
-<wire x1="142.24" y1="109.22" x2="142.24" y2="101.6" width="0.1524" layer="91"/>
-<junction x="142.24" y="101.6"/>
-</segment>
-<segment>
+<wire x1="139.7" y1="101.6" x2="127" y2="101.6" width="0.1524" layer="91"/>
+<wire x1="139.7" y1="109.22" x2="139.7" y2="101.6" width="0.1524" layer="91"/>
+<junction x="139.7" y="101.6"/>
+</segment>
+<segment>
