File: cad/epaper.sch (EAGLE design)
At the start: 4 parts

Commit message: tweak
Parts:
- added U$2, U$3: FIDUCIAL, adafruit:FIDUCIAL
Changed lines of the file:
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@@
 <?xml version="1.0" encoding="utf-8"?>
 <!DOCTYPE eagle SYSTEM "eagle.dtd">
-<eagle version="7.1.0">
+<eagle version="7.2.0">
 <drawing>
 <settings>
@@
 <layer number="97" name="Info" color="7" fill="1" visible="yes" active="yes"/>
 <layer number="98" name="Guide" color="6" fill="1" visible="yes" active="yes"/>
+<layer number="99" name="SpiceOrder" color="7" fill="1" visible="no" active="no"/>
 <layer number="100" name="Muster" color="7" fill="1" visible="yes" active="yes"/>
 <layer number="101" name="Hidden" color="15" fill="1" visible="yes" active="yes"/>
@@
 <layer number="111" name="LPC17xx" color="7" fill="1" visible="yes" active="yes"/>
 <layer number="112" name="tSilk" color="7" fill="1" visible="yes" active="yes"/>
+<layer number="113" name="ReferenceLS" color="7" fill="1" visible="no" active="no"/>
 <layer number="116" name="Patch_BOT" color="7" fill="1" visible="yes" active="yes"/>
+<layer number="118" name="Rect_Pads" color="7" fill="1" visible="no" active="no"/>
 <layer number="121" name="_tsilk" color="7" fill="1" visible="yes" active="yes"/>
 <layer number="122" name="_bsilk" color="7" fill="1" visible="yes" active="yes"/>
@@
 <layer number="223" name="223bmp" color="24" fill="1" visible="no" active="no"/>
 <layer number="224" name="224bmp" color="25" fill="1" visible="no" active="no"/>
+<layer number="231" name="Eagle3D_PG1" color="7" fill="1" visible="no" active="no"/>
+<layer number="232" name="Eagle3D_PG2" color="7" fill="1" visible="no" active="no"/>
+<layer number="233" name="Eagle3D_PG3" color="7" fill="1" visible="no" active="no"/>
 <layer number="248" name="Housing" color="7" fill="1" visible="yes" active="yes"/>
 <layer number="249" name="Edge" color="7" fill="1" visible="yes" active="yes"/>
@@
 <part name="VCC1" library="jaw" deviceset="PWR-VCC" device=""/>
 <part name="U$1" library="jaw" deviceset="ROBOTMAN-LOGO" device=""/>
+<part name="U$2" library="adafruit" deviceset="FIDUCIAL" device=""/>
+<part name="U$3" library="adafruit" deviceset="FIDUCIAL" device=""/>
 </parts>
 <sheets>
@@
 <instance part="VCC1" gate="G$1" x="40.64" y="60.96"/>
 <instance part="U$1" gate="G$1" x="7.62" y="5.08"/>
+<instance part="U$2" gate="G$1" x="20.32" y="7.62"/>
+<instance part="U$3" gate="G$1" x="27.94" y="7.62"/>
 </instances>
 <busses>

Commit message: silk text
Parts:
- U$1: value ROBOTMAN-LOGO -> ROBOTMAN-LOGO2; device jaw:ROBOTMAN-LOGO -> jaw:ROBOTMAN-LOGO2
Changed lines of the file:
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@@
 <part name="GND1" library="jaw" deviceset="PWR-GND" device=""/>
 <part name="VCC1" library="jaw" deviceset="PWR-VCC" device=""/>
-<part name="U$1" library="jaw" deviceset="ROBOTMAN-LOGO" device=""/>
+<part name="U$1" library="jaw" deviceset="ROBOTMAN-LOGO" device="2" value="ROBOTMAN-LOGO2"/>
 <part name="U$2" library="adafruit" deviceset="FIDUCIAL" device=""/>
 <part name="U$3" library="adafruit" deviceset="FIDUCIAL" device=""/>

Commit message: embiggen connector
Parts:
- removed CN1: (no value), jaw:HEADER-2X4
- added CONN2: HEADER-5X2-PTH, jaw:HEADER-5X2-PTH
- C1: value (none) -> .1u
Connections:
- new net N$12: CONN2.9
- new net N$19: CONN2.10
- net DPYCS: now also CONN2.7; no longer CN1.P$7
- net DPYDC: now also CONN2.6; no longer CN1.P$6
- net GND: now also CONN2.8; no longer CN1.P$8
- net NRST: now also CONN2.2; no longer CN1.P$2
- net SPIMISO: now also CONN2.3; no longer CN1.P$3
- net SPIMOSI: now also CONN2.5; no longer CN1.P$5
- net SPISCK: now also CONN2.4; no longer CN1.P$4
- net VCC: now also CONN2.1; no longer CN1.P$1
Changed lines of the file:
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@@
 <layer number="56" name="wert" color="7" fill="1" visible="no" active="no"/>
 <layer number="57" name="tCAD" color="7" fill="1" visible="no" active="no"/>
+<layer number="59" name="tCarbon" color="7" fill="1" visible="no" active="no"/>
+<layer number="60" name="bCarbon" color="7" fill="1" visible="no" active="no"/>
 <layer number="90" name="Modules" color="5" fill="1" visible="yes" active="yes"/>
 <layer number="91" name="Nets" color="2" fill="1" visible="yes" active="yes"/>
@@
 <layer number="127" name="_tValues" color="7" fill="1" visible="yes" active="yes"/>
 <layer number="128" name="_bValues" color="7" fill="1" visible="yes" active="yes"/>
+<layer number="129" name="Mask" color="7" fill="1" visible="yes" active="yes"/>
 <layer number="131" name="prix" color="7" fill="1" visible="yes" active="yes"/>
 <layer number="132" name="test" color="7" fill="1" visible="yes" active="yes"/>
@@
 <layer number="223" name="223bmp" color="24" fill="1" visible="no" active="no"/>
 <layer number="224" name="224bmp" color="25" fill="1" visible="no" active="no"/>
+<layer number="225" name="225bmp" color="7" fill="1" visible="yes" active="yes"/>
+<layer number="226" name="226bmp" color="7" fill="1" visible="yes" active="yes"/>
+<layer number="227" name="227bmp" color="7" fill="1" visible="yes" active="yes"/>
+<layer number="228" name="228bmp" color="7" fill="1" visible="yes" active="yes"/>
+<layer number="229" name="229bmp" color="7" fill="1" visible="yes" active="yes"/>
+<layer number="230" name="230bmp" color="7" fill="1" visible="yes" active="yes"/>
 <layer number="231" name="Eagle3D_PG1" color="7" fill="1" visible="no" active="no"/>
 <layer number="232" name="Eagle3D_PG2" color="7" fill="1" visible="no" active="no"/>
@@
 <layer number="251" name="SMDround" color="7" fill="1" visible="yes" active="yes"/>
 <layer number="254" name="cooling" color="7" fill="1" visible="yes" active="yes"/>
+<layer number="255" name="routoute" color="7" fill="1" visible="yes" active="yes"/>
 </layers>
 <schematic xreflabel="%F%N/%S.%C%R" xrefpart="/%S.%C%R">
@@
 </classes>
 <parts>
-<part name="CN1" library="jaw" deviceset="HEADER-2X4" device=""/>
-<part name="GND24" library="jaw" deviceset="PWR-GND" device=""/>
-<part name="VCC20" library="jaw" deviceset="PWR-VCC" device=""/>
 <part name="SV1" library="jaw" deviceset="MA10-1" device="-M05/FFC"/>
-<part name="C1" library="jaw" deviceset="C" device="0603"/>
+<part name="C1" library="jaw" deviceset="C" device="0603" value=".1u"/>
 <part name="GND1" library="jaw" deviceset="PWR-GND" device=""/>
 <part name="VCC1" library="jaw" deviceset="PWR-VCC" device=""/>
@@
 <part name="U$2" library="adafruit" deviceset="FIDUCIAL" device=""/>
 <part name="U$3" library="adafruit" deviceset="FIDUCIAL" device=""/>
+<part name="CONN2" library="jaw" deviceset="HEADER-5X2" device="-PTH"/>
+<part name="VCC2" library="jaw" deviceset="PWR-VCC" device=""/>
+<part name="GND3" library="jaw" deviceset="PWR-GND" device=""/>
 </parts>
 <sheets>
@@
 </plain>
 <instances>
-<instance part="CN1" gate="A" x="35.56" y="22.86"/>
-<instance part="GND24" gate="G$1" x="48.26" y="17.78"/>
-<instance part="VCC20" gate="G$1" x="20.32" y="30.48"/>
 <instance part="SV1" gate="1" x="111.76" y="33.02" rot="R180"/>
 <instance part="C1" gate="G$1" x="40.64" y="55.88" rot="R180"/>
@@
 <instance part="U$2" gate="G$1" x="20.32" y="7.62"/>
 <instance part="U$3" gate="G$1" x="27.94" y="7.62"/>
+<instance part="CONN2" gate="G$1" x="43.18" y="22.86"/>
+<instance part="VCC2" gate="G$1" x="33.02" y="35.56"/>
+<instance part="GND3" gate="G$1" x="58.42" y="22.86"/>
 </instances>
 <busses>
@@
 <net name="GND" class="0">
 <segment>
-<pinref part="CN1" gate="A" pin="P$8"/>
-<pinref part="GND24" gate="G$1" pin="GND"/>
-<wire x1="48.26" y1="20.32" x2="40.64" y2="20.32" width="0.1524" layer="91"/>
-</segment>
-<segment>
 <pinref part="C1" gate="G$1" pin="P$1"/>
 <pinref part="GND1" gate="G$1" pin="GND"/>
@@
 <label x="91.44" y="25.4" size="1.27" layer="95"/>
 </segment>
+<segment>
+<pinref part="CONN2" gate="G$1" pin="8"/>
+<wire x1="50.8" y1="25.4" x2="53.34" y2="25.4" width="0.1524" layer="91"/>
+<pinref part="GND3" gate="G$1" pin="GND"/>
+<wire x1="53.34" y1="25.4" x2="58.42" y2="25.4" width="0.1524" layer="91"/>
+</segment>
 </net>
 <net name="VCC" class="0">
-<segment>
-<pinref part="CN1" gate="A" pin="P$1"/>
-<pinref part="VCC20" gate="G$1" pin="VCC"/>
-<wire x1="20.32" y1="27.94" x2="33.02" y2="27.94" width="0.1524" layer="91"/>
-</segment>
 <segment>
 <pinref part="C1" gate="G$1" pin="P$2"/>
@@
 <label x="91.44" y="27.94" size="1.27" layer="95"/>
 </segment>
+<segment>
+<pinref part="CONN2" gate="G$1" pin="1"/>
+<wire x1="35.56" y1="33.02" x2="33.02" y2="33.02" width="0.1524" layer="91"/>
+<pinref part="VCC2" gate="G$1" pin="VCC"/>
+</segment>
 </net>
 <net name="NRST" class="0">
 <segment>
-<pinref part="CN1" gate="A" pin="P$2"/>
-<wire x1="40.64" y1="27.94" x2="48.26" y2="27.94" width="0.1524" layer="91"/>
-<label x="48.26" y="27.94" size="1.778" layer="95"/>
+<pinref part="CONN2" gate="G$1" pin="2"/>
+<wire x1="50.8" y1="33.02" x2="53.34" y2="33.02" width="0.1524" layer="91"/>
+<label x="53.34" y="33.02" size="1.778" layer="95"/>
 </segment>
 </net>
 <net name="DPYDC" class="0">
 <segment>
-<pinref part="CN1" gate="A" pin="P$6"/>
-<wire x1="40.64" y1="22.86" x2="48.26" y2="22.86" width="0.1524" layer="91"/>
-<label x="48.26" y="22.86" size="1.778" layer="95"/>
+<pinref part="CONN2" gate="G$1" pin="6"/>
+<wire x1="50.8" y1="27.94" x2="53.34" y2="27.94" width="0.1524" layer="91"/>
+<label x="53.34" y="27.94" size="1.778" layer="95"/>
 </segment>
 </net>
 <net name="SPISCK" class="0">
-<segment>
-<pinref part="CN1" gate="A" pin="P$4"/>
-<wire x1="40.64" y1="25.4" x2="48.26" y2="25.4" width="0.1524" layer="91"/>
-<label x="48.26" y="25.4" size="1.778" layer="95"/>
-</segment>
 <segment>
 <pinref part="SV1" gate="1" pin="1"/>
@@
 <label x="91.44" y="43.18" size="1.27" layer="95"/>
 </segment>
+<segment>
+<pinref part="CONN2" gate="G$1" pin="4"/>
+<wire x1="50.8" y1="30.48" x2="53.34" y2="30.48" width="0.1524" layer="91"/>
+<label x="53.34" y="30.48" size="1.778" layer="95"/>
+</segment>
 </net>
 <net name="SPIMISO" class="0">
 <segment>
-<pinref part="CN1" gate="A" pin="P$3"/>
-<wire x1="33.02" y1="25.4" x2="30.48" y2="25.4" width="0.1524" layer="91"/>
-<label x="20.32" y="25.4" size="1.778" layer="95"/>
+<pinref part="CONN2" gate="G$1" pin="3"/>
+<wire x1="35.56" y1="30.48" x2="33.02" y2="30.48" width="0.1524" layer="91"/>
+<label x="22.86" y="30.48" size="1.778" layer="95"/>
 </segment>
 </net>
 <net name="SPIMOSI" class="0">
-<segment>
-<pinref part="CN1" gate="A" pin="P$5"/>
-<wire x1="33.02" y1="22.86" x2="30.48" y2="22.86" width="0.1524" layer="91"/>
-<label x="20.32" y="22.86" size="1.778" layer="95"/>
-</segment>
 <segment>
 <pinref part="SV1" gate="1" pin="2"/>
@@
 <label x="91.44" y="40.64" size="1.27" layer="95"/>
 </segment>
+<segment>
+<pinref part="CONN2" gate="G$1" pin="5"/>
+<wire x1="35.56" y1="27.94" x2="33.02" y2="27.94" width="0.1524" layer="91"/>
+<label x="22.86" y="27.94" size="1.778" layer="95"/>
+</segment>
 </net>
 <net name="DPYCS" class="0">
-<segment>
-<pinref part="CN1" gate="A" pin="P$7"/>
-<wire x1="33.02" y1="20.32" x2="30.48" y2="20.32" width="0.1524" layer="91"/>
-<label x="22.86" y="20.32" size="1.778" layer="95"/>
-</segment>
 <segment>
 <pinref part="SV1" gate="1" pin="3"/>
@@
 <label x="91.44" y="38.1" size="1.27" layer="95"/>
 </segment>
+<segment>
+<pinref part="CONN2" gate="G$1" pin="7"/>
+<wire x1="35.56" y1="25.4" x2="33.02" y2="25.4" width="0.1524" layer="91"/>
+<label x="22.86" y="25.4" size="1.778" layer="95"/>
+</segment>
 </net>
 <net name="N$4" class="0">
@@
 </segment>
 </net>
+<net name="N$12" class="0">
+<segment>
+<pinref part="CONN2" gate="G$1" pin="9"/>
+<wire x1="35.56" y1="22.86" x2="33.02" y2="22.86" width="0.1524" layer="91"/>
+</segment>
+</net>
+<net name="N$19" class="0">
+<segment>
+<pinref part="CONN2" gate="G$1" pin="10"/>
+<wire x1="50.8" y1="22.86" x2="53.34" y2="22.86" width="0.1524" layer="91"/>
+</segment>
+</net>
