File: cad/oled.brd (EAGLE design)
At the start: 17.5 x 21.5 mm, 3 parts, among them CN2 MA12-1

Commit message: tweak
Parts:
- added U$1, U$2: FIDUCIAL, adafruit:FIDUCIAL_1MM
Other:
- board size 17.5 x 21.5 mm -> 17.1 x 21.5 mm
- board text added: "OLED 128x32"
Changed lines of the file:
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@@
 <?xml version="1.0" encoding="utf-8"?>
 <!DOCTYPE eagle SYSTEM "eagle.dtd">
-<eagle version="7.1.0">
+<eagle version="7.2.0">
 <drawing>
 <settings>
@@
 <layers>
 <layer number="1" name="Top" color="4" fill="1" visible="yes" active="yes"/>
+<layer number="2" name="Route2" color="1" fill="3" visible="no" active="yes"/>
+<layer number="3" name="Route3" color="4" fill="3" visible="no" active="yes"/>
+<layer number="14" name="Route14" color="1" fill="6" visible="no" active="yes"/>
+<layer number="15" name="Route15" color="4" fill="6" visible="no" active="yes"/>
 <layer number="16" name="Bottom" color="1" fill="1" visible="yes" active="yes"/>
 <layer number="17" name="Pads" color="2" fill="1" visible="yes" active="yes"/>
@@
 <layer number="54" name="bGND_GNDA" color="7" fill="1" visible="no" active="no"/>
 <layer number="56" name="wert" color="7" fill="1" visible="no" active="no"/>
+<layer number="57" name="tCAD" color="7" fill="1" visible="no" active="no"/>
 <layer number="91" name="Nets" color="2" fill="1" visible="no" active="no"/>
 <layer number="92" name="Busses" color="1" fill="1" visible="no" active="no"/>
@@
 <layer number="97" name="Info" color="7" fill="1" visible="no" active="no"/>
 <layer number="98" name="Guide" color="6" fill="1" visible="no" active="no"/>
+<layer number="99" name="SpiceOrder" color="7" fill="1" visible="no" active="no"/>
 <layer number="100" name="Muster" color="7" fill="1" visible="yes" active="yes"/>
 <layer number="101" name="Hidden" color="15" fill="1" visible="yes" active="yes"/>
@@
 <layer number="111" name="LPC17xx" color="7" fill="1" visible="yes" active="yes"/>
 <layer number="112" name="tSilk" color="7" fill="1" visible="yes" active="yes"/>
+<layer number="113" name="ReferenceLS" color="7" fill="1" visible="no" active="no"/>
 <layer number="116" name="Patch_BOT" color="7" fill="1" visible="yes" active="yes"/>
+<layer number="118" name="Rect_Pads" color="7" fill="1" visible="no" active="no"/>
 <layer number="121" name="_tsilk" color="7" fill="1" visible="yes" active="yes"/>
 <layer number="122" name="_bsilk" color="7" fill="1" visible="yes" active="yes"/>
@@
 <layer number="132" name="test" color="7" fill="1" visible="yes" active="yes"/>
 <layer number="144" name="Drill_legend" color="7" fill="1" visible="yes" active="yes"/>
+<layer number="150" name="Notes" color="7" fill="1" visible="no" active="yes"/>
 <layer number="151" name="HeatSink" color="7" fill="1" visible="yes" active="yes"/>
 <layer number="152" name="_bDocu" color="7" fill="1" visible="yes" active="yes"/>
+<layer number="153" name="FabDoc1" color="6" fill="1" visible="no" active="no"/>
+<layer number="154" name="FabDoc2" color="2" fill="1" visible="no" active="no"/>
+<layer number="155" name="FabDoc3" color="7" fill="15" visible="no" active="no"/>
 <layer number="199" name="Contour" color="7" fill="1" visible="yes" active="yes"/>
 <layer number="200" name="200bmp" color="7" fill="1" visible="yes" active="yes"/>
@@
 <layer number="223" name="223bmp" color="24" fill="1" visible="no" active="no"/>
 <layer number="224" name="224bmp" color="25" fill="1" visible="no" active="no"/>
+<layer number="231" name="Eagle3D_PG1" color="7" fill="1" visible="no" active="no"/>
+<layer number="232" name="Eagle3D_PG2" color="7" fill="1" visible="no" active="no"/>
+<layer number="233" name="Eagle3D_PG3" color="7" fill="1" visible="no" active="no"/>
 <layer number="248" name="Housing" color="7" fill="1" visible="yes" active="yes"/>
 <layer number="249" name="Edge" color="7" fill="1" visible="yes" active="yes"/>
@@
 <board>
 <plain>
-<wire x1="19.5" y1="54.5" x2="4" y2="54.5" width="0" layer="20"/>
+<wire x1="4" y1="33" x2="15.5" y2="33" width="0" layer="20"/>
+<wire x1="15.5" y1="33" x2="16.5" y2="34" width="0" layer="20" curve="90"/>
+<wire x1="16.5" y1="34" x2="16.5" y2="44.2" width="0" layer="20"/>
+<wire x1="16.5" y1="44.2" x2="20.1" y2="44.2" width="0" layer="20"/>
+<wire x1="20.1" y1="44.2" x2="20.1" y2="54.5" width="0" layer="20"/>
+<wire x1="20.1" y1="54.5" x2="4" y2="54.5" width="0" layer="20"/>
 <wire x1="4" y1="54.5" x2="3" y2="53.5" width="0" layer="20" curve="90"/>
 <wire x1="3" y1="53.5" x2="3" y2="34" width="0" layer="20"/>
 <wire x1="3" y1="34" x2="4" y2="33" width="0" layer="20" curve="90"/>
-<wire x1="4" y1="33" x2="13.2" y2="33" width="0" layer="20"/>
-<wire x1="13.2" y1="33" x2="14.2" y2="34" width="0" layer="20" curve="90"/>
-<wire x1="14.2" y1="34" x2="14.2" y2="43.2" width="0" layer="20"/>
-<wire x1="14.2" y1="43.2" x2="15.2" y2="44.2" width="0" layer="20" curve="-90"/>
-<wire x1="15.2" y1="44.2" x2="19.5" y2="44.2" width="0" layer="20"/>
-<wire x1="19.5" y1="44.2" x2="20.5" y2="45.2" width="0" layer="20" curve="90"/>
-<wire x1="20.5" y1="45.2" x2="20.5" y2="53.5" width="0" layer="20"/>
-<wire x1="20.5" y1="53.5" x2="19.5" y2="54.5" width="0" layer="20" curve="90"/>
 <text x="14" y="54" size="1" layer="22" ratio="10" rot="MR270">JAW 2015-03</text>
 <text x="12.5" y="54" size="1.1" layer="22" ratio="10" rot="MR270">mini32/oled</text>
+<text x="16" y="34" size="1" layer="21" ratio="10" rot="R90">OLED 128x32</text>
 </plain>
 <attributes>
@@
 <attribute name="VALUE" x="7.258" y="41.314" size="1.27" layer="28" font="vector" ratio="10" rot="MR0"/>
 </element>
+<element name="U$1" library="adafruit" package="FIDUCIAL_1MM" value="FIDUCIAL" x="14.5" y="35" rot="MR0"/>
+<element name="U$2" library="adafruit" package="FIDUCIAL_1MM" value="FIDUCIAL" x="4.5" y="53" rot="MR0"/>
 </elements>
 <signals>

Commit message: silk text
Other:
- board text added: "www.amiketo.com"
- board text removed: "mini32/oled"
Changed lines of the file:
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@@
 <wire x1="3" y1="53.5" x2="3" y2="34" width="0" layer="20"/>
 <wire x1="3" y1="34" x2="4" y2="33" width="0" layer="20" curve="90"/>
-<text x="14" y="54" size="1" layer="22" ratio="10" rot="MR270">JAW 2015-03</text>
-<text x="12.5" y="54" size="1.1" layer="22" ratio="10" rot="MR270">mini32/oled</text>
+<text x="14" y="54" size="1.25" layer="22" ratio="10" rot="MR270">JAW 2015-03</text>
+<text x="12.3" y="54" size="1.05" layer="22" ratio="10" rot="MR270">www.amiketo.com</text>
 <text x="16" y="34" size="1" layer="21" ratio="10" rot="R90">OLED 128x32</text>
 </plain>
@@
 </element>
 <element name="CN2" library="jaw" package="M05-1X12-RA" value="MA12-1" x="8.6" y="39.35" smashed="yes" rot="MR0">
-<attribute name="NAME" x="10.3" y="36.75" size="1.27" layer="26" rot="MR0"/>
+<attribute name="NAME" x="10.3" y="36.75" size="1.27" layer="26" rot="MR0" display="off"/>
 </element>
 <element name="C1" library="jaw" package="SMD0603" value=".1u" x="5.48" y="43.6" smashed="yes" rot="MR0">

Commit message: embiggen connector
Parts:
- removed CN1: (no value), jaw:HEADER-2X04
- added CONN2: HEADER-5X2-PTH, jaw:HEADER-5X2-PTH
Connections:
- new net N$12: CONN2.9
- new net N$19: CONN2.10
- net DPYCS: now also CONN2.7; no longer CN1.7
- net DPYDC: now also CONN2.6; no longer CN1.6
- net GND: now also CONN2.8; no longer CN1.8
- net NRST: now also CONN2.2; no longer CN1.2
- net SPIMISO: now also CONN2.3; no longer CN1.3
- net SPIMOSI: now also CONN2.5; no longer CN1.5
- net SPISCK: now also CONN2.4; no longer CN1.4
- net VCC: now also CONN2.1; no longer CN1.1
Other:
- outline, holes or cut-outs redrawn
- board text added: "JAW 2015-04"
- board text removed: "JAW 2015-03"
