File: cad/oled.sch (EAGLE design)
At the start: 3 parts, among them CN2 MA12-1

Commit message: tweak
Parts:
- added U$1, U$2: FIDUCIAL, adafruit:FIDUCIAL
Changed lines of the file:
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@@
 <?xml version="1.0" encoding="utf-8"?>
 <!DOCTYPE eagle SYSTEM "eagle.dtd">
-<eagle version="7.1.0">
+<eagle version="7.2.0">
 <drawing>
 <settings>
@@
 <layers>
 <layer number="1" name="Top" color="4" fill="1" visible="no" active="no"/>
+<layer number="2" name="Route2" color="1" fill="3" visible="no" active="no"/>
+<layer number="3" name="Route3" color="4" fill="3" visible="no" active="no"/>
+<layer number="14" name="Route14" color="1" fill="6" visible="no" active="no"/>
+<layer number="15" name="Route15" color="4" fill="6" visible="no" active="no"/>
 <layer number="16" name="Bottom" color="1" fill="1" visible="no" active="no"/>
 <layer number="17" name="Pads" color="2" fill="1" visible="no" active="no"/>
@@
 <layer number="54" name="bGND_GNDA" color="7" fill="1" visible="no" active="no"/>
 <layer number="56" name="wert" color="7" fill="1" visible="no" active="no"/>
+<layer number="57" name="tCAD" color="7" fill="1" visible="no" active="no"/>
 <layer number="91" name="Nets" color="2" fill="1" visible="yes" active="yes"/>
 <layer number="92" name="Busses" color="1" fill="1" visible="yes" active="yes"/>
@@
 <layer number="97" name="Info" color="7" fill="1" visible="yes" active="yes"/>
 <layer number="98" name="Guide" color="6" fill="1" visible="yes" active="yes"/>
+<layer number="99" name="SpiceOrder" color="7" fill="1" visible="no" active="no"/>
 <layer number="100" name="Muster" color="7" fill="1" visible="yes" active="yes"/>
 <layer number="101" name="Hidden" color="15" fill="1" visible="yes" active="yes"/>
@@
 <layer number="111" name="LPC17xx" color="7" fill="1" visible="yes" active="yes"/>
 <layer number="112" name="tSilk" color="7" fill="1" visible="yes" active="yes"/>
+<layer number="113" name="ReferenceLS" color="7" fill="1" visible="no" active="no"/>
 <layer number="116" name="Patch_BOT" color="7" fill="1" visible="yes" active="yes"/>
+<layer number="118" name="Rect_Pads" color="7" fill="1" visible="no" active="no"/>
 <layer number="121" name="_tsilk" color="7" fill="1" visible="yes" active="yes"/>
 <layer number="122" name="_bsilk" color="7" fill="1" visible="yes" active="yes"/>
@@
 <layer number="132" name="test" color="7" fill="1" visible="yes" active="yes"/>
 <layer number="144" name="Drill_legend" color="7" fill="1" visible="yes" active="yes"/>
+<layer number="150" name="Notes" color="7" fill="1" visible="no" active="yes"/>
 <layer number="151" name="HeatSink" color="7" fill="1" visible="yes" active="yes"/>
 <layer number="152" name="_bDocu" color="7" fill="1" visible="yes" active="yes"/>
+<layer number="153" name="FabDoc1" color="6" fill="1" visible="no" active="no"/>
+<layer number="154" name="FabDoc2" color="2" fill="1" visible="no" active="no"/>
+<layer number="155" name="FabDoc3" color="7" fill="15" visible="no" active="no"/>
 <layer number="199" name="Contour" color="7" fill="1" visible="yes" active="yes"/>
 <layer number="200" name="200bmp" color="7" fill="1" visible="yes" active="yes"/>
@@
 <layer number="223" name="223bmp" color="24" fill="1" visible="no" active="no"/>
 <layer number="224" name="224bmp" color="25" fill="1" visible="no" active="no"/>
+<layer number="231" name="Eagle3D_PG1" color="7" fill="1" visible="no" active="no"/>
+<layer number="232" name="Eagle3D_PG2" color="7" fill="1" visible="no" active="no"/>
+<layer number="233" name="Eagle3D_PG3" color="7" fill="1" visible="no" active="no"/>
 <layer number="248" name="Housing" color="7" fill="1" visible="yes" active="yes"/>
 <layer number="249" name="Edge" color="7" fill="1" visible="yes" active="yes"/>
@@
 <part name="VCC1" library="jaw" deviceset="PWR-VCC" device=""/>
 <part name="GND1" library="jaw" deviceset="PWR-GND" device=""/>
+<part name="U$1" library="adafruit" deviceset="FIDUCIAL" device=""/>
+<part name="U$2" library="adafruit" deviceset="FIDUCIAL" device=""/>
 </parts>
 <sheets>
@@
 <instance part="VCC1" gate="G$1" x="83.82" y="66.04"/>
 <instance part="GND1" gate="G$1" x="83.82" y="48.26"/>
+<instance part="U$1" gate="G$1" x="142.24" y="10.16"/>
+<instance part="U$2" gate="G$1" x="149.86" y="10.16"/>
 </instances>
 <busses>

Commit message: embiggen connector
Parts:
- removed CN1: (no value), jaw:HEADER-2X4
- added CONN2: HEADER-5X2-PTH, jaw:HEADER-5X2-PTH
Connections:
- new net N$12: CONN2.9
- new net N$19: CONN2.10
- net DPYCS: now also CONN2.7; no longer CN1.P$7
- net DPYDC: now also CONN2.6; no longer CN1.P$6
- net GND: now also CONN2.8; no longer CN1.P$8
- net NRST: now also CONN2.2; no longer CN1.P$2
- net SPIMISO: now also CONN2.3; no longer CN1.P$3
- net SPIMOSI: now also CONN2.5; no longer CN1.P$5
- net SPISCK: now also CONN2.4; no longer CN1.P$4
- net VCC: now also CONN2.1; no longer CN1.P$1
Changed lines of the file:
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@@
 <layer number="56" name="wert" color="7" fill="1" visible="no" active="no"/>
 <layer number="57" name="tCAD" color="7" fill="1" visible="no" active="no"/>
+<layer number="59" name="tCarbon" color="7" fill="1" visible="no" active="no"/>
+<layer number="60" name="bCarbon" color="7" fill="1" visible="no" active="no"/>
+<layer number="90" name="Modules" color="5" fill="1" visible="yes" active="yes"/>
 <layer number="91" name="Nets" color="2" fill="1" visible="yes" active="yes"/>
 <layer number="92" name="Busses" color="1" fill="1" visible="yes" active="yes"/>
@@
 <layer number="127" name="_tValues" color="7" fill="1" visible="yes" active="yes"/>
 <layer number="128" name="_bValues" color="7" fill="1" visible="yes" active="yes"/>
+<layer number="129" name="Mask" color="7" fill="1" visible="yes" active="yes"/>
 <layer number="131" name="prix" color="7" fill="1" visible="yes" active="yes"/>
 <layer number="132" name="test" color="7" fill="1" visible="yes" active="yes"/>
@@
 <layer number="223" name="223bmp" color="24" fill="1" visible="no" active="no"/>
 <layer number="224" name="224bmp" color="25" fill="1" visible="no" active="no"/>
+<layer number="225" name="225bmp" color="7" fill="1" visible="yes" active="yes"/>
+<layer number="226" name="226bmp" color="7" fill="1" visible="yes" active="yes"/>
+<layer number="227" name="227bmp" color="7" fill="1" visible="yes" active="yes"/>
+<layer number="228" name="228bmp" color="7" fill="1" visible="yes" active="yes"/>
+<layer number="229" name="229bmp" color="7" fill="1" visible="yes" active="yes"/>
+<layer number="230" name="230bmp" color="7" fill="1" visible="yes" active="yes"/>
 <layer number="231" name="Eagle3D_PG1" color="7" fill="1" visible="no" active="no"/>
 <layer number="232" name="Eagle3D_PG2" color="7" fill="1" visible="no" active="no"/>
@@
 <layer number="251" name="SMDround" color="7" fill="1" visible="yes" active="yes"/>
 <layer number="254" name="cooling" color="7" fill="1" visible="yes" active="yes"/>
+<layer number="255" name="routoute" color="7" fill="1" visible="yes" active="yes"/>
 </layers>
 <schematic xreflabel="%F%N/%S.%C%R" xrefpart="/%S.%C%R">
@@
 </classes>
 <parts>
-<part name="CN1" library="jaw" deviceset="HEADER-2X4" device=""/>
-<part name="GND24" library="jaw" deviceset="PWR-GND" device=""/>
-<part name="VCC20" library="jaw" deviceset="PWR-VCC" device=""/>
 <part name="CN2" library="jaw" deviceset="MA12-1" device=""/>
 <part name="C1" library="jaw" deviceset="C" device="0603" value=".1u"/>
@@
 <part name="U$1" library="adafruit" deviceset="FIDUCIAL" device=""/>
 <part name="U$2" library="adafruit" deviceset="FIDUCIAL" device=""/>
+<part name="CONN2" library="jaw" deviceset="HEADER-5X2" device="-PTH"/>
+<part name="VCC2" library="jaw" deviceset="PWR-VCC" device=""/>
+<part name="GND3" library="jaw" deviceset="PWR-GND" device=""/>
 </parts>
 <sheets>
@@
 </plain>
 <instances>
-<instance part="CN1" gate="A" x="38.1" y="27.94"/>
-<instance part="GND24" gate="G$1" x="50.8" y="22.86"/>
-<instance part="VCC20" gate="G$1" x="22.86" y="35.56"/>
 <instance part="CN2" gate="G$1" x="111.76" y="33.02"/>
 <instance part="C1" gate="G$1" x="83.82" y="55.88"/>
@@
 <instance part="U$1" gate="G$1" x="142.24" y="10.16"/>
 <instance part="U$2" gate="G$1" x="149.86" y="10.16"/>
+<instance part="CONN2" gate="G$1" x="40.64" y="7.62"/>
+<instance part="VCC2" gate="G$1" x="30.48" y="20.32"/>
+<instance part="GND3" gate="G$1" x="55.88" y="7.62"/>
 </instances>
 <busses>
@@
 <net name="GND" class="0">
 <segment>
-<pinref part="CN1" gate="A" pin="P$8"/>
-<pinref part="GND24" gate="G$1" pin="GND"/>
-<wire x1="50.8" y1="25.4" x2="43.18" y2="25.4" width="0.1524" layer="91"/>
-</segment>
-<segment>
 <pinref part="CN2" gate="G$1" pin="P1"/>
 <wire x1="104.14" y1="45.72" x2="99.06" y2="45.72" width="0.1524" layer="91"/>
@@
 <label x="96.52" y="25.4" size="1.778" layer="95"/>
 </segment>
+<segment>
+<pinref part="CONN2" gate="G$1" pin="8"/>
+<wire x1="48.26" y1="10.16" x2="50.8" y2="10.16" width="0.1524" layer="91"/>
+<pinref part="GND3" gate="G$1" pin="GND"/>
+<wire x1="50.8" y1="10.16" x2="55.88" y2="10.16" width="0.1524" layer="91"/>
+</segment>
 </net>
 <net name="VCC" class="0">
-<segment>
-<pinref part="CN1" gate="A" pin="P$1"/>
-<pinref part="VCC20" gate="G$1" pin="VCC"/>
-<wire x1="22.86" y1="33.02" x2="35.56" y2="33.02" width="0.1524" layer="91"/>
-</segment>
 <segment>
 <pinref part="CN2" gate="G$1" pin="P10"/>
@@
 <pinref part="VCC1" gate="G$1" pin="VCC"/>
 </segment>
+<segment>
+<pinref part="CONN2" gate="G$1" pin="1"/>
+<wire x1="33.02" y1="17.78" x2="30.48" y2="17.78" width="0.1524" layer="91"/>
+<pinref part="VCC2" gate="G$1" pin="VCC"/>
+</segment>
 </net>
 <net name="NRST" class="0">
-<segment>
-<pinref part="CN1" gate="A" pin="P$2"/>
-<wire x1="43.18" y1="33.02" x2="50.8" y2="33.02" width="0.1524" layer="91"/>
-<label x="50.8" y="33.02" size="1.778" layer="95"/>
-</segment>
 <segment>
 <pinref part="CN2" gate="G$1" pin="P6"/>
@@
 <label x="96.52" y="33.02" size="1.778" layer="95"/>
 </segment>
+<segment>
+<pinref part="CONN2" gate="G$1" pin="2"/>
+<wire x1="48.26" y1="17.78" x2="50.8" y2="17.78" width="0.1524" layer="91"/>
+<label x="50.8" y="17.78" size="1.778" layer="95"/>
+</segment>
 </net>
 <net name="DPYDC" class="0">
-<segment>
-<pinref part="CN1" gate="A" pin="P$6"/>
-<wire x1="43.18" y1="27.94" x2="50.8" y2="27.94" width="0.1524" layer="91"/>
-<label x="50.8" y="27.94" size="1.778" layer="95"/>
-</segment>
 <segment>
 <pinref part="CN2" gate="G$1" pin="P5"/>
@@
 <label x="96.52" y="35.56" size="1.778" layer="95"/>
 </segment>
+<segment>
+<pinref part="CONN2" gate="G$1" pin="6"/>
+<wire x1="48.26" y1="12.7" x2="50.8" y2="12.7" width="0.1524" layer="91"/>
+<label x="50.8" y="12.7" size="1.778" layer="95"/>
+</segment>
 </net>
 <net name="SPISCK" class="0">
-<segment>
-<pinref part="CN1" gate="A" pin="P$4"/>
-<wire x1="43.18" y1="30.48" x2="50.8" y2="30.48" width="0.1524" layer="91"/>
-<label x="50.8" y="30.48" size="1.778" layer="95"/>
-</segment>
 <segment>
 <pinref part="CN2" gate="G$1" pin="P4"/>
@@
 <label x="96.52" y="38.1" size="1.778" layer="95"/>
 </segment>
+<segment>
+<pinref part="CONN2" gate="G$1" pin="4"/>
+<wire x1="48.26" y1="15.24" x2="50.8" y2="15.24" width="0.1524" layer="91"/>
+<label x="50.8" y="15.24" size="1.778" layer="95"/>
+</segment>
 </net>
 <net name="SPIMISO" class="0">
 <segment>
-<pinref part="CN1" gate="A" pin="P$3"/>
-<wire x1="35.56" y1="30.48" x2="33.02" y2="30.48" width="0.1524" layer="91"/>
-<label x="22.86" y="30.48" size="1.778" layer="95"/>
+<pinref part="CONN2" gate="G$1" pin="3"/>
+<wire x1="33.02" y1="15.24" x2="30.48" y2="15.24" width="0.1524" layer="91"/>
+<label x="20.32" y="15.24" size="1.778" layer="95"/>
 </segment>
 </net>
 <net name="SPIMOSI" class="0">
-<segment>
-<pinref part="CN1" gate="A" pin="P$5"/>
-<wire x1="35.56" y1="27.94" x2="33.02" y2="27.94" width="0.1524" layer="91"/>
-<label x="22.86" y="27.94" size="1.778" layer="95"/>
-</segment>
 <segment>
 <pinref part="CN2" gate="G$1" pin="P3"/>
@@
 <label x="96.52" y="40.64" size="1.778" layer="95"/>
 </segment>
+<segment>
+<pinref part="CONN2" gate="G$1" pin="5"/>
+<wire x1="33.02" y1="12.7" x2="30.48" y2="12.7" width="0.1524" layer="91"/>
+<label x="20.32" y="12.7" size="1.778" layer="95"/>
+</segment>
 </net>
 <net name="DPYCS" class="0">
-<segment>
-<pinref part="CN1" gate="A" pin="P$7"/>
-<wire x1="35.56" y1="25.4" x2="33.02" y2="25.4" width="0.1524" layer="91"/>
-<label x="25.4" y="25.4" size="1.778" layer="95"/>
-</segment>
 <segment>
 <pinref part="CN2" gate="G$1" pin="P7"/>
@@
 <label x="96.52" y="30.48" size="1.778" layer="95"/>
 </segment>
-</net>
+<segment>
+<pinref part="CONN2" gate="G$1" pin="7"/>
+<wire x1="33.02" y1="10.16" x2="30.48" y2="10.16" width="0.1524" layer="91"/>
+<label x="20.32" y="10.16" size="1.778" layer="95"/>
+</segment>
+</net>
+<net name="N$12" class="0">
+<segment>
+<pinref part="CONN2" gate="G$1" pin="9"/>
+<wire x1="33.02" y1="7.62" x2="30.48" y2="7.62" width="0.1524" layer="91"/>
+</segment>
+</net>
+<net name="N$19" class="0">
+<segment>
+<pinref part="CONN2" gate="G$1" pin="10"/>
+<wire x1="48.26" y1="7.62" x2="50.8" y2="7.62" width="0.1524" layer="91"/>
+</segment>
+</net>
