File: cad/oled2.sch (EAGLE design)
At the start: 10 parts

Commit message: tweak
Parts:
- added U$1, U$2: FIDUCIAL, adafruit:FIDUCIAL
Changed lines of the file:
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@@
 <?xml version="1.0" encoding="utf-8"?>
 <!DOCTYPE eagle SYSTEM "eagle.dtd">
-<eagle version="7.1.0">
+<eagle version="7.2.0">
 <drawing>
 <settings>
@@
 <setting verticaltext="up"/>
 </settings>
-<grid distance="0.1" unitdist="inch" unit="inch" style="lines" multiple="1" display="yes" altdistance="0.01" altunitdist="inch" altunit="inch"/>
+<grid distance="0.1" unitdist="inch" unit="inch" style="lines" multiple="1" display="no" altdistance="0.01" altunitdist="inch" altunit="inch"/>
 <layers>
 <layer number="1" name="Top" color="4" fill="1" visible="no" active="no"/>
@@
 <layer number="54" name="bGND_GNDA" color="7" fill="1" visible="no" active="no"/>
 <layer number="56" name="wert" color="7" fill="1" visible="no" active="no"/>
+<layer number="57" name="tCAD" color="7" fill="1" visible="no" active="no"/>
 <layer number="91" name="Nets" color="2" fill="1" visible="yes" active="yes"/>
 <layer number="92" name="Busses" color="1" fill="1" visible="yes" active="yes"/>
@@
 <layer number="97" name="Info" color="7" fill="1" visible="yes" active="yes"/>
 <layer number="98" name="Guide" color="6" fill="1" visible="yes" active="yes"/>
+<layer number="99" name="SpiceOrder" color="7" fill="1" visible="no" active="no"/>
 <layer number="100" name="Muster" color="7" fill="1" visible="yes" active="yes"/>
 <layer number="101" name="Hidden" color="15" fill="1" visible="yes" active="yes"/>
@@
 <layer number="111" name="LPC17xx" color="7" fill="1" visible="yes" active="yes"/>
 <layer number="112" name="tSilk" color="7" fill="1" visible="yes" active="yes"/>
+<layer number="113" name="ReferenceLS" color="7" fill="1" visible="no" active="no"/>
 <layer number="116" name="Patch_BOT" color="7" fill="1" visible="yes" active="yes"/>
+<layer number="118" name="Rect_Pads" color="7" fill="1" visible="no" active="no"/>
 <layer number="121" name="_tsilk" color="7" fill="1" visible="yes" active="yes"/>
 <layer number="122" name="_bsilk" color="7" fill="1" visible="yes" active="yes"/>
@@
 <layer number="132" name="test" color="7" fill="1" visible="yes" active="yes"/>
 <layer number="144" name="Drill_legend" color="7" fill="1" visible="yes" active="yes"/>
+<layer number="150" name="Notes" color="7" fill="1" visible="no" active="yes"/>
 <layer number="151" name="HeatSink" color="7" fill="1" visible="yes" active="yes"/>
 <layer number="152" name="_bDocu" color="7" fill="1" visible="yes" active="yes"/>
+<layer number="153" name="FabDoc1" color="6" fill="1" visible="no" active="no"/>
+<layer number="154" name="FabDoc2" color="2" fill="1" visible="no" active="no"/>
+<layer number="155" name="FabDoc3" color="7" fill="15" visible="no" active="no"/>
 <layer number="199" name="Contour" color="7" fill="1" visible="yes" active="yes"/>
 <layer number="200" name="200bmp" color="7" fill="1" visible="yes" active="yes"/>
@@
 <layer number="223" name="223bmp" color="24" fill="1" visible="no" active="no"/>
 <layer number="224" name="224bmp" color="25" fill="1" visible="no" active="no"/>
+<layer number="231" name="Eagle3D_PG1" color="7" fill="1" visible="no" active="no"/>
+<layer number="232" name="Eagle3D_PG2" color="7" fill="1" visible="no" active="no"/>
+<layer number="233" name="Eagle3D_PG3" color="7" fill="1" visible="no" active="no"/>
 <layer number="248" name="Housing" color="7" fill="1" visible="yes" active="yes"/>
 <layer number="249" name="Edge" color="7" fill="1" visible="yes" active="yes"/>
@@
 <part name="C7" library="jaw" deviceset="C" device="0603" value="10u"/>
 <part name="R1" library="jaw" deviceset="R" device="0603" value="390k"/>
+<part name="U$1" library="adafruit" deviceset="FIDUCIAL" device=""/>
+<part name="U$2" library="adafruit" deviceset="FIDUCIAL" device=""/>
 </parts>
 <sheets>
@@
 <instance part="C7" gate="G$1" x="76.2" y="55.88"/>
 <instance part="R1" gate="G$1" x="116.84" y="20.32"/>
+<instance part="U$1" gate="G$1" x="170.18" y="7.62"/>
+<instance part="U$2" gate="G$1" x="177.8" y="7.62"/>
 </instances>
 <busses>

Commit message: silk text
Parts:
- added LOGO1: OSHW-LOGOS, Sparkfun-Aesthetics:OSHW-LOGOS
- added U$3: ROBOTMAN-LOGO2, jaw:ROBOTMAN-LOGO2
Changed lines of the file:
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@@
 <layer number="56" name="wert" color="7" fill="1" visible="no" active="no"/>
 <layer number="57" name="tCAD" color="7" fill="1" visible="no" active="no"/>
+<layer number="59" name="tCarbon" color="7" fill="1" visible="no" active="no"/>
+<layer number="60" name="bCarbon" color="7" fill="1" visible="no" active="no"/>
+<layer number="90" name="Modules" color="5" fill="1" visible="yes" active="yes"/>
 <layer number="91" name="Nets" color="2" fill="1" visible="yes" active="yes"/>
 <layer number="92" name="Busses" color="1" fill="1" visible="yes" active="yes"/>
@@
 <layer number="127" name="_tValues" color="7" fill="1" visible="yes" active="yes"/>
 <layer number="128" name="_bValues" color="7" fill="1" visible="yes" active="yes"/>
+<layer number="129" name="Mask" color="7" fill="1" visible="yes" active="yes"/>
 <layer number="131" name="prix" color="7" fill="1" visible="yes" active="yes"/>
 <layer number="132" name="test" color="7" fill="1" visible="yes" active="yes"/>
@@
 <layer number="223" name="223bmp" color="24" fill="1" visible="no" active="no"/>
 <layer number="224" name="224bmp" color="25" fill="1" visible="no" active="no"/>
+<layer number="225" name="225bmp" color="7" fill="1" visible="yes" active="yes"/>
+<layer number="226" name="226bmp" color="7" fill="1" visible="yes" active="yes"/>
+<layer number="227" name="227bmp" color="7" fill="1" visible="yes" active="yes"/>
+<layer number="228" name="228bmp" color="7" fill="1" visible="yes" active="yes"/>
+<layer number="229" name="229bmp" color="7" fill="1" visible="yes" active="yes"/>
+<layer number="230" name="230bmp" color="7" fill="1" visible="yes" active="yes"/>
 <layer number="231" name="Eagle3D_PG1" color="7" fill="1" visible="no" active="no"/>
 <layer number="232" name="Eagle3D_PG2" color="7" fill="1" visible="no" active="no"/>
@@
 <layer number="251" name="SMDround" color="7" fill="1" visible="yes" active="yes"/>
 <layer number="254" name="cooling" color="7" fill="1" visible="yes" active="yes"/>
+<layer number="255" name="routoute" color="7" fill="1" visible="yes" active="yes"/>
 </layers>
 <schematic xreflabel="%F%N/%S.%C%R" xrefpart="/%S.%C%R">
@@
 <part name="U$1" library="adafruit" deviceset="FIDUCIAL" device=""/>
 <part name="U$2" library="adafruit" deviceset="FIDUCIAL" device=""/>
+<part name="U$3" library="jaw" deviceset="ROBOTMAN-LOGO" device="2"/>
+<part name="LOGO1" library="Sparkfun-Aesthetics" deviceset="OSHW-LOGO" device="S"/>
 </parts>
 <sheets>
@@
 <instance part="U$1" gate="G$1" x="170.18" y="7.62"/>
 <instance part="U$2" gate="G$1" x="177.8" y="7.62"/>
+<instance part="U$3" gate="G$1" x="187.96" y="7.62"/>
+<instance part="LOGO1" gate="G$1" x="180.34" y="22.86"/>
 </instances>
 <busses>

Commit message: connector
Parts:
- removed CN1: (no value), jaw:HEADER-2X4
- added CONN2: HEADER-5X2-PTH, jaw:HEADER-5X2-PTH
Connections:
- new net N$12: CONN2.9
- new net N$19: CONN2.10
- net DPYCS: now also CONN2.7; no longer CN1.P$7
- net DPYDC: now also CONN2.6; no longer CN1.P$6
- net GND: now also CONN2.8; no longer CN1.P$8
- net NRST: now also CONN2.2; no longer CN1.P$2
- net SPIMISO: now also CONN2.3; no longer CN1.P$3
- net SPIMOSI: now also CONN2.5; no longer CN1.P$5
- net SPISCK: now also CONN2.4; no longer CN1.P$4
- net VCC: now also CONN2.1; no longer CN1.P$1
Other:
- note added: "0.96", 128x64 pixel, ssd1306 based monochrome OLED, ebay special"
- note removed: "0.96", 96x64 pixel, ssd1306 based monochrome OLED, ebay special"
Changed lines of the file:
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@@
 <setting verticaltext="up"/>
 </settings>
-<grid distance="0.1" unitdist="inch" unit="inch" style="lines" multiple="1" display="no" altdistance="0.01" altunitdist="inch" altunit="inch"/>
+<grid distance="0.1" unitdist="inch" unit="inch" style="lines" multiple="1" display="yes" altdistance="0.01" altunitdist="inch" altunit="inch"/>
 <layers>
 <layer number="1" name="Top" color="4" fill="1" visible="no" active="no"/>
@@
 </classes>
 <parts>
-<part name="CN1" library="jaw" deviceset="HEADER-2X4" device=""/>
-<part name="GND24" library="jaw" deviceset="PWR-GND" device=""/>
-<part name="VCC20" library="jaw" deviceset="PWR-VCC" device=""/>
 <part name="C1" library="jaw" deviceset="C" device="0603" value=".1u"/>
 <part name="VCC1" library="jaw" deviceset="PWR-VCC" device=""/>
@@
 <part name="U$3" library="jaw" deviceset="ROBOTMAN-LOGO" device="2"/>
 <part name="LOGO1" library="Sparkfun-Aesthetics" deviceset="OSHW-LOGO" device="S"/>
+<part name="CONN2" library="jaw" deviceset="HEADER-5X2" device="-PTH"/>
+<part name="VCC2" library="jaw" deviceset="PWR-VCC" device=""/>
+<part name="GND3" library="jaw" deviceset="PWR-GND" device=""/>
 </parts>
 <sheets>
@@
 <text x="142.24" y="17.78" size="1.27" layer="97">VCOM</text>
 <text x="142.24" y="15.24" size="1.27" layer="97">VCC</text>
-<text x="25.4" y="81.28" size="2.54" layer="97">0.96", 96x64 pixel, ssd1306 based
+<text x="25.4" y="81.28" size="2.54" layer="97">0.96", 128x64 pixel, ssd1306 based
 monochrome OLED, ebay special</text>
 </plain>
 <instances>
-<instance part="CN1" gate="A" x="38.1" y="27.94"/>
-<instance part="GND24" gate="G$1" x="50.8" y="22.86"/>
-<instance part="VCC20" gate="G$1" x="22.86" y="35.56"/>
 <instance part="C1" gate="G$1" x="83.82" y="55.88"/>
 <instance part="VCC1" gate="G$1" x="83.82" y="66.04"/>
@@
 <instance part="U$3" gate="G$1" x="187.96" y="7.62"/>
 <instance part="LOGO1" gate="G$1" x="180.34" y="22.86"/>
+<instance part="CONN2" gate="G$1" x="40.64" y="40.64"/>
+<instance part="VCC2" gate="G$1" x="30.48" y="53.34"/>
+<instance part="GND3" gate="G$1" x="55.88" y="40.64"/>
 </instances>
 <busses>
@@
 <nets>
 <net name="GND" class="0">
-<segment>
-<pinref part="CN1" gate="A" pin="P$8"/>
-<pinref part="GND24" gate="G$1" pin="GND"/>
-<wire x1="50.8" y1="25.4" x2="43.18" y2="25.4" width="0.1524" layer="91"/>
-</segment>
 <segment>
 <pinref part="C1" gate="G$1" pin="P$2"/>
@@
 <junction x="99.06" y="17.78"/>
 </segment>
+<segment>
+<pinref part="CONN2" gate="G$1" pin="8"/>
+<wire x1="48.26" y1="43.18" x2="50.8" y2="43.18" width="0.1524" layer="91"/>
+<pinref part="GND3" gate="G$1" pin="GND"/>
+<wire x1="50.8" y1="43.18" x2="55.88" y2="43.18" width="0.1524" layer="91"/>
+</segment>
 </net>
 <net name="VCC" class="0">
-<segment>
-<pinref part="CN1" gate="A" pin="P$1"/>
-<pinref part="VCC20" gate="G$1" pin="VCC"/>
-<wire x1="22.86" y1="33.02" x2="35.56" y2="33.02" width="0.1524" layer="91"/>
-</segment>
 <segment>
 <pinref part="C1" gate="G$1" pin="P$1"/>
@@
 <label x="124.46" y="71.12" size="1.27" layer="95"/>
 </segment>
+<segment>
+<pinref part="CONN2" gate="G$1" pin="1"/>
+<wire x1="33.02" y1="50.8" x2="30.48" y2="50.8" width="0.1524" layer="91"/>
+<pinref part="VCC2" gate="G$1" pin="VCC"/>
+</segment>
 </net>
 <net name="NRST" class="0">
-<segment>
-<pinref part="CN1" gate="A" pin="P$2"/>
-<wire x1="43.18" y1="33.02" x2="50.8" y2="33.02" width="0.1524" layer="91"/>
-<label x="50.8" y="33.02" size="1.778" layer="95"/>
-</segment>
 <segment>
 <pinref part="CONN1" gate="G$1" pin="14"/>
@@
 <label x="124.46" y="50.8" size="1.27" layer="95"/>
 </segment>
+<segment>
+<pinref part="CONN2" gate="G$1" pin="2"/>
+<wire x1="48.26" y1="50.8" x2="50.8" y2="50.8" width="0.1524" layer="91"/>
+<label x="50.8" y="50.8" size="1.778" layer="95"/>
+</segment>
 </net>
 <net name="DPYDC" class="0">
-<segment>
-<pinref part="CN1" gate="A" pin="P$6"/>
-<wire x1="43.18" y1="27.94" x2="50.8" y2="27.94" width="0.1524" layer="91"/>
-<label x="50.8" y="27.94" size="1.778" layer="95"/>
-</segment>
 <segment>
 <pinref part="CONN1" gate="G$1" pin="15"/>
@@
 <label x="124.46" y="48.26" size="1.27" layer="95"/>
 </segment>
+<segment>
+<pinref part="CONN2" gate="G$1" pin="6"/>
+<wire x1="48.26" y1="45.72" x2="50.8" y2="45.72" width="0.1524" layer="91"/>
+<label x="50.8" y="45.72" size="1.778" layer="95"/>
+</segment>
 </net>
 <net name="SPISCK" class="0">
-<segment>
-<pinref part="CN1" gate="A" pin="P$4"/>
-<wire x1="43.18" y1="30.48" x2="50.8" y2="30.48" width="0.1524" layer="91"/>
-<label x="50.8" y="30.48" size="1.778" layer="95"/>
-</segment>
 <segment>
 <pinref part="CONN1" gate="G$1" pin="18"/>
@@
 <label x="124.46" y="40.64" size="1.27" layer="95"/>
 </segment>
+<segment>
+<pinref part="CONN2" gate="G$1" pin="4"/>
+<wire x1="48.26" y1="48.26" x2="50.8" y2="48.26" width="0.1524" layer="91"/>
+<label x="50.8" y="48.26" size="1.778" layer="95"/>
+</segment>
 </net>
 <net name="SPIMISO" class="0">
 <segment>
-<pinref part="CN1" gate="A" pin="P$3"/>
-<wire x1="35.56" y1="30.48" x2="33.02" y2="30.48" width="0.1524" layer="91"/>
-<label x="22.86" y="30.48" size="1.778" layer="95"/>
+<pinref part="CONN2" gate="G$1" pin="3"/>
+<wire x1="33.02" y1="48.26" x2="30.48" y2="48.26" width="0.1524" layer="91"/>
+<label x="20.32" y="48.26" size="1.778" layer="95"/>
 </segment>
 </net>
 <net name="SPIMOSI" class="0">
-<segment>
-<pinref part="CN1" gate="A" pin="P$5"/>
-<wire x1="35.56" y1="27.94" x2="33.02" y2="27.94" width="0.1524" layer="91"/>
-<label x="22.86" y="27.94" size="1.778" layer="95"/>
-</segment>
 <segment>
 <pinref part="CONN1" gate="G$1" pin="19"/>
@@
 <label x="124.46" y="38.1" size="1.27" layer="95"/>
 </segment>
+<segment>
+<pinref part="CONN2" gate="G$1" pin="5"/>
+<wire x1="33.02" y1="45.72" x2="30.48" y2="45.72" width="0.1524" layer="91"/>
+<label x="20.32" y="45.72" size="1.778" layer="95"/>
+</segment>
 </net>
 <net name="DPYCS" class="0">
-<segment>
-<pinref part="CN1" gate="A" pin="P$7"/>
-<wire x1="35.56" y1="25.4" x2="33.02" y2="25.4" width="0.1524" layer="91"/>
-<label x="25.4" y="25.4" size="1.778" layer="95"/>
-</segment>
 <segment>
 <pinref part="CONN1" gate="G$1" pin="13"/>
 <wire x1="137.16" y1="53.34" x2="129.54" y2="53.34" width="0.1524" layer="91"/>
 <label x="124.46" y="53.34" size="1.27" layer="95"/>
+</segment>
+<segment>
+<pinref part="CONN2" gate="G$1" pin="7"/>
+<wire x1="33.02" y1="43.18" x2="30.48" y2="43.18" width="0.1524" layer="91"/>
+<label x="20.32" y="43.18" size="1.778" layer="95"/>
 </segment>
 </net>
@@
 </segment>
 </net>
+<net name="N$12" class="0">
+<segment>
+<pinref part="CONN2" gate="G$1" pin="9"/>
+<wire x1="33.02" y1="40.64" x2="30.48" y2="40.64" width="0.1524" layer="91"/>
+</segment>
+</net>
+<net name="N$19" class="0">
+<segment>
+<pinref part="CONN2" gate="G$1" pin="10"/>
+<wire x1="48.26" y1="40.64" x2="50.8" y2="40.64" width="0.1524" layer="91"/>
+</segment>
+</net>

Commit message: embiggen connector
Other:
- note added: "0.96", 128x64 pixel, ssd1306 based monochrome OLED"
- note removed: "0.96", 128x64 pixel, ssd1306 based monochrome OLED, ebay special"
- moved on the sheet: C1, C7
Changed lines of the file:
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@@
 <setting verticaltext="up"/>
 </settings>
-<grid distance="0.1" unitdist="inch" unit="inch" style="lines" multiple="1" display="yes" altdistance="0.01" altunitdist="inch" altunit="inch"/>
+<grid distance="0.1" unitdist="inch" unit="inch" style="lines" multiple="1" display="no" altdistance="0.01" altunitdist="inch" altunit="inch"/>
 <layers>
 <layer number="1" name="Top" color="4" fill="1" visible="no" active="no"/>
@@
 <text x="142.24" y="15.24" size="1.27" layer="97">VCC</text>
 <text x="25.4" y="81.28" size="2.54" layer="97">0.96", 128x64 pixel, ssd1306 based
-monochrome OLED, ebay special</text>
+monochrome OLED</text>
 </plain>
 <instances>
-<instance part="C1" gate="G$1" x="83.82" y="55.88"/>
-<instance part="VCC1" gate="G$1" x="83.82" y="66.04"/>
-<instance part="GND1" gate="G$1" x="83.82" y="48.26"/>
+<instance part="C1" gate="G$1" x="78.74" y="12.7"/>
+<instance part="VCC1" gate="G$1" x="78.74" y="22.86"/>
+<instance part="GND1" gate="G$1" x="78.74" y="5.08"/>
 <instance part="CONN1" gate="G$1" x="137.16" y="45.72"/>
 <instance part="C2" gate="G$1" x="116.84" y="81.28" rot="R90"/>
@@
 <instance part="C6" gate="G$1" x="106.68" y="17.78" rot="R90"/>
 <instance part="GND2" gate="G$1" x="99.06" y="5.08"/>
-<instance part="C7" gate="G$1" x="76.2" y="55.88"/>
+<instance part="C7" gate="G$1" x="71.12" y="12.7"/>
 <instance part="R1" gate="G$1" x="116.84" y="20.32"/>
 <instance part="U$1" gate="G$1" x="170.18" y="7.62"/>
@@
 <segment>
 <pinref part="C1" gate="G$1" pin="P$2"/>
-<wire x1="83.82" y1="53.34" x2="83.82" y2="50.8" width="0.1524" layer="91"/>
+<wire x1="78.74" y1="10.16" x2="78.74" y2="7.62" width="0.1524" layer="91"/>
 <pinref part="GND1" gate="G$1" pin="GND"/>
 <pinref part="C7" gate="G$1" pin="P$2"/>
-<wire x1="76.2" y1="53.34" x2="83.82" y2="53.34" width="0.1524" layer="91"/>
-<junction x="83.82" y="53.34"/>
+<wire x1="71.12" y1="10.16" x2="78.74" y2="10.16" width="0.1524" layer="91"/>
+<junction x="78.74" y="10.16"/>
 </segment>
 <segment>
@@
 <segment>
 <pinref part="C1" gate="G$1" pin="P$1"/>
-<wire x1="83.82" y1="60.96" x2="83.82" y2="63.5" width="0.1524" layer="91"/>
+<wire x1="78.74" y1="17.78" x2="78.74" y2="20.32" width="0.1524" layer="91"/>
 <pinref part="VCC1" gate="G$1" pin="VCC"/>
 <pinref part="C7" gate="G$1" pin="P$1"/>
-<wire x1="83.82" y1="60.96" x2="76.2" y2="60.96" width="0.1524" layer="91"/>
-<junction x="83.82" y="60.96"/>
+<wire x1="78.74" y1="17.78" x2="71.12" y2="17.78" width="0.1524" layer="91"/>
+<junction x="78.74" y="17.78"/>
 </segment>
 <segment>
@@
 <net name="NRST" class="0">
 <segment>
+<pinref part="CONN2" gate="G$1" pin="2"/>
+<wire x1="48.26" y1="50.8" x2="50.8" y2="50.8" width="0.1524" layer="91"/>
+<label x="50.8" y="50.8" size="1.778" layer="95"/>
+</segment>
+<segment>
 <pinref part="CONN1" gate="G$1" pin="14"/>
 <wire x1="137.16" y1="50.8" x2="129.54" y2="50.8" width="0.1524" layer="91"/>
 <label x="124.46" y="50.8" size="1.27" layer="95"/>
 </segment>
-<segment>
-<pinref part="CONN2" gate="G$1" pin="2"/>
-<wire x1="48.26" y1="50.8" x2="50.8" y2="50.8" width="0.1524" layer="91"/>
-<label x="50.8" y="50.8" size="1.778" layer="95"/>
-</segment>
 </net>
