File: cad/oled2.brd (EAGLE design)
At the start: 28.5 x 24.2 mm, 10 parts

Commit message: tweak
Parts:
- added U$1, U$2: FIDUCIAL, adafruit:FIDUCIAL_1MM
- moved CONN1 5.00 mm to (50.0, 22.5)
Routing:
- net GND: track 87.3 -> 102.1 mm, vias 1 -> 18
- net VCC: track 22.6 -> 32.6 mm
- net N$4: track 6.04 -> 11.0 mm
- net N$27: track 4.61 -> 9.61 mm
- net SPISCK: track 25.7 -> 30.7 mm
- net N$5: track 3.97 -> 8.97 mm
- net N$29: track 5.83 -> 10.8 mm
- net N$28: track 3.80 -> 8.80 mm
- net DPYDC: track 21.1 -> 26.1 mm
- net N$6: track 6.06 -> 11.1 mm
- net N$3: track 3.80 -> 8.80 mm
- net DPYCS: track 14.0 -> 19.0 mm
- net SPIMOSI: track 23.1 -> 28.1 mm
- net NRST: track 23.8 -> 28.8 mm
- added copper zone on layer 1, net GND
- added copper zone on layer 16, net GND
- added copper zone on layer 16, net N$2
Other:
- board size 28.5 x 24.2 mm -> 28.5 x 29.2 mm
- board text added: "oled 128x64"

Commit message: silk text
Parts:
- added LOGO1: OSHW-LOGOS, Sparkfun-Aesthetics:OSHW-LOGO-S
- added U$3: ROBOTMAN-LOGO2, jaw:ROBOTMAN-LOGO2
- moved U$2 10.3 mm to (36.5, 6.50)
Routing:
- net GND: track 102.1 -> 87.3 mm, vias 18 -> 19
Other:
- board text added: "JAW 2015-04"
- board text added: "www.amiketo.com"
- board text removed: "JAW 2015-03"
- board text removed: "mini32/oled-0.96"
Changed lines of the file:
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@@
 <grid distance="0.1" unitdist="mm" unit="mm" style="lines" multiple="5" display="yes" altdistance="0.025" altunitdist="inch" altunit="inch"/>
 <layers>
-<layer number="1" name="Top" color="4" fill="1" visible="yes" active="yes"/>
+<layer number="1" name="Top" color="4" fill="1" visible="no" active="yes"/>
 <layer number="2" name="Route2" color="1" fill="3" visible="no" active="no"/>
 <layer number="3" name="Route3" color="4" fill="3" visible="no" active="no"/>
@@
 <layer number="19" name="Unrouted" color="6" fill="1" visible="yes" active="yes"/>
 <layer number="20" name="Dimension" color="15" fill="1" visible="yes" active="yes"/>
-<layer number="21" name="tPlace" color="7" fill="1" visible="yes" active="yes"/>
+<layer number="21" name="tPlace" color="7" fill="1" visible="no" active="yes"/>
 <layer number="22" name="bPlace" color="7" fill="1" visible="yes" active="yes"/>
 <layer number="23" name="tOrigins" color="15" fill="1" visible="yes" active="yes"/>
@@
 <layer number="56" name="wert" color="7" fill="1" visible="no" active="no"/>
 <layer number="57" name="tCAD" color="7" fill="1" visible="no" active="no"/>
+<layer number="59" name="tCarbon" color="7" fill="1" visible="no" active="no"/>
+<layer number="60" name="bCarbon" color="7" fill="1" visible="no" active="no"/>
+<layer number="90" name="Modules" color="5" fill="1" visible="no" active="no"/>
 <layer number="91" name="Nets" color="2" fill="1" visible="no" active="no"/>
 <layer number="92" name="Busses" color="1" fill="1" visible="no" active="no"/>
@@
 <layer number="127" name="_tValues" color="7" fill="1" visible="yes" active="yes"/>
 <layer number="128" name="_bValues" color="7" fill="1" visible="yes" active="yes"/>
+<layer number="129" name="Mask" color="7" fill="1" visible="yes" active="yes"/>
 <layer number="131" name="prix" color="7" fill="1" visible="yes" active="yes"/>
 <layer number="132" name="test" color="7" fill="1" visible="yes" active="yes"/>
@@
 <layer number="223" name="223bmp" color="24" fill="1" visible="no" active="no"/>
 <layer number="224" name="224bmp" color="25" fill="1" visible="no" active="no"/>
+<layer number="225" name="225bmp" color="7" fill="1" visible="yes" active="yes"/>
+<layer number="226" name="226bmp" color="7" fill="1" visible="yes" active="yes"/>
+<layer number="227" name="227bmp" color="7" fill="1" visible="yes" active="yes"/>
+<layer number="228" name="228bmp" color="7" fill="1" visible="yes" active="yes"/>
+<layer number="229" name="229bmp" color="7" fill="1" visible="yes" active="yes"/>
+<layer number="230" name="230bmp" color="7" fill="1" visible="yes" active="yes"/>
 <layer number="231" name="Eagle3D_PG1" color="7" fill="1" visible="no" active="no"/>
 <layer number="232" name="Eagle3D_PG2" color="7" fill="1" visible="no" active="no"/>
@@
 <layer number="251" name="SMDround" color="7" fill="1" visible="yes" active="yes"/>
 <layer number="254" name="cooling" color="7" fill="1" visible="yes" active="yes"/>
+<layer number="255" name="routoute" color="7" fill="1" visible="yes" active="yes"/>
 </layers>
 <board>
@@
 <wire x1="53.3" y1="4" x2="53.3" y2="0.8" width="0" layer="20"/>
 <wire x1="53.3" y1="0.8" x2="63.5" y2="0.8" width="0" layer="20"/>
-<text x="51" y="6.5" size="1.5" layer="22" ratio="10" rot="MR0">JAW 2015-03</text>
-<text x="51" y="4.7" size="1.1" layer="22" ratio="10" rot="MR0">mini32/oled-0.96</text>
+<text x="53.1" y="7" size="1.5" layer="22" ratio="10" rot="MR0">JAW 2015-04</text>
+<text x="53" y="5" size="1.25" layer="22" ratio="10" rot="MR0">www.amiketo.com</text>
 <text x="37.5" y="4.5" size="1.5" layer="21" ratio="10">oled 128x64</text>
 </plain>
@@
 </element>
 <element name="U$1" library="adafruit" package="FIDUCIAL_1MM" value="FIDUCIAL" x="61.5" y="27.5" rot="MR0"/>
-<element name="U$2" library="adafruit" package="FIDUCIAL_1MM" value="FIDUCIAL" x="39" y="16.5" rot="MR0"/>
+<element name="U$2" library="adafruit" package="FIDUCIAL_1MM" value="FIDUCIAL" x="36.5" y="6.5" rot="MR0"/>
+<element name="U$3" library="jaw" package="ROBOTMAN-LOGO2" value="ROBOTMAN-LOGO2" x="47.8" y="15.1" rot="MR0"/>
+<element name="LOGO1" library="Sparkfun-Aesthetics" package="OSHW-LOGO-S" value="OSHW-LOGOS" x="56" y="7" rot="MR0"/>
 </elements>
 <signals>
@@
 <wire x1="58.8" y1="26.1" x2="54.9" y2="26.1" width="0.35" layer="16"/>
 <wire x1="38.3" y1="12.2" x2="37.9142125" y2="12.2" width="0.35" layer="16"/>
-<wire x1="37.9142125" y1="12.2" x2="37.20710625" y2="12.49289375" width="0.35" layer="16" curve="-45"/>
-<wire x1="37.20710625" y1="12.49289375" x2="37.19289375" y2="12.50710625" width="0.35" layer="16"/>
-<wire x1="37.19289375" y1="12.50710625" x2="36.9" y2="13.2142125" width="0.35" layer="16" curve="-45"/>
-<wire x1="36.9" y1="13.2142125" x2="36.9" y2="25.1" width="0.35" layer="16"/>
-<wire x1="36.9" y1="25.1" x2="37.9" y2="26.1" width="0.35" layer="16" curve="-90"/>
 <wire x1="37.9" y1="26.1" x2="39.5" y2="26.1" width="0.35" layer="16"/>
 <contactref element="R1" pad="1"/>
@@
 <via x="60.9" y="18.2" extent="1-16" drill="0.35"/>
 <via x="55.3" y="18.9" extent="1-16" drill="0.35"/>
+<via x="52.8" y="15.5" extent="1-16" drill="0.35"/>
 </signal>
 <signal name="VCC">
@@
 <contactref element="CONN1" pad="6"/>
 <contactref element="C7" pad="1"/>
-<wire x1="56.3" y1="16.2" x2="56.3" y2="16.4" width="0.25" layer="16"/>
-<wire x1="56.3" y1="16.4" x2="56.3" y2="22.5" width="0.25" layer="16"/>
-<wire x1="62.2" y1="4.58" x2="62.21" y2="4.57" width="0.25" layer="16"/>
+<wire x1="56.3" y1="15.45" x2="56.3" y2="22.5" width="0.25" layer="16"/>
 <wire x1="54.2" y1="22.5" x2="54.2" y2="15.45" width="0.25" layer="16"/>
 <wire x1="54.2" y1="15.45" x2="54.45" y2="15.2" width="0.25" layer="16" curve="90"/>
@@
 <wire x1="62.2" y1="8.371571875" x2="62.2" y2="4.58" width="0.25" layer="16"/>
 <wire x1="62.2" y1="4.58" x2="62.21" y2="4.57" width="0.25" layer="16"/>
-<wire x1="56.3" y1="16.2" x2="56.3" y2="16.4" width="0.35" layer="16"/>
-<wire x1="56.3" y1="16.4" x2="56.3" y2="15.45" width="0.25" layer="16"/>
 <wire x1="56.3" y1="15.45" x2="56.05" y2="15.2" width="0.25" layer="16" curve="-90"/>
 <wire x1="56.05" y1="15.2" x2="55.6" y2="15.2" width="0.25" layer="16"/>

Commit message: connector
Parts:
- removed CN1: (no value), jaw:HEADER-2X04
- added CONN2: HEADER-5X2-PTH, jaw:HEADER-5X2-PTH
- moved C1 0.20 mm to (54.8, 13.9)
- moved C7 0.20 mm to (54.8, 12.1)
Connections:
- new net N$12: CONN2.9
- new net N$19: CONN2.10
- net DPYCS: now also CONN2.7; no longer CN1.7
- net DPYDC: now also CONN2.6; no longer CN1.6
- net GND: now also CONN2.8; no longer CN1.8
- net NRST: now also CONN2.2; no longer CN1.2
- net SPIMISO: now also CONN2.3; no longer CN1.3
- net SPIMOSI: now also CONN2.5; no longer CN1.5
- net SPISCK: now also CONN2.4; no longer CN1.4
- net VCC: now also CONN2.1; no longer CN1.1
Routing:
- net GND: track 87.3 -> 65.7 mm
Other:
- outline, holes or cut-outs redrawn

Commit message: embiggen connector
Parts:
- moved CONN1 3.00 mm to (50.0, 19.5)
- moved U$1 3.00 mm to (61.5, 24.5)
- moved U$3 2.78 mm to (50.0, 13.4), flipped to the top
- moved C7 1.35 mm to (53.8, 13.0), turned to 270 degrees
- moved C1 1.27 mm to (55.7, 13.0), turned to 270 degrees
Routing:
- net GND: track 65.7 -> 85.0 mm, vias 19 -> 21
- net SPIMOSI: track 28.1 -> 22.8 mm
- net NRST: track 28.8 -> 24.2 mm
- net SPISCK: track 30.7 -> 26.3 mm
- net DPYDC: track 26.1 -> 22.1 mm
- net DPYCS: track 19.0 -> 15.6 mm
- net N$4: track 11.0 -> 8.04 mm
- net N$29: track 10.8 -> 7.83 mm
- net N$28: track 8.80 -> 5.80 mm
- net N$5: track 8.97 -> 5.97 mm
- net N$27: track 9.61 -> 6.61 mm
- net N$3: track 8.80 -> 5.80 mm
- net N$6: track 11.1 -> 8.06 mm
- net VCC: track 31.9 -> 29.6 mm, vias 0 -> 1
Other:
- board size 28.5 x 29.2 mm -> 28.5 x 26.2 mm
