File: cad/amiketo_2hm.brd (EAGLE design)
At the start: 35 x 35 mm, 56 parts, among them CN1 MICROSD-EJECT, CN2 DO NOT PLACE, Q1 IRLML6344TRPBF, Q2 DMP2035U-7, SW2 SWITCHKMR211, SW3 SWITCHKMR211, U1 STM32F411/48, U2 LIS3DH, X1 12MHz, X2 32k768

Commit message: tweak
Parts:
- CN2: device jaw:HEADER-3X2-PTH -> jaw:HEADER-3X2-POGO
Routing:
- net GND: vias 41 -> 42
Changed lines of the file:
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@@
 <layers>
 <layer number="1" name="Top" color="4" fill="1" visible="yes" active="yes"/>
-<layer number="2" name="Route2" color="5" fill="1" visible="no" active="yes"/>
+<layer number="2" name="Route2" color="5" fill="1" visible="yes" active="yes"/>
 <layer number="3" name="Route3" color="4" fill="3" visible="no" active="no"/>
 <layer number="14" name="Route14" color="1" fill="6" visible="no" active="no"/>
-<layer number="15" name="Route15" color="1" fill="1" visible="no" active="yes"/>
-<layer number="16" name="Bottom" color="6" fill="1" visible="no" active="yes"/>
+<layer number="15" name="Route15" color="1" fill="1" visible="yes" active="yes"/>
+<layer number="16" name="Bottom" color="6" fill="1" visible="yes" active="yes"/>
 <layer number="17" name="Pads" color="2" fill="1" visible="yes" active="yes"/>
 <layer number="18" name="Vias" color="2" fill="1" visible="yes" active="yes"/>
@@
 <attribute name="VALUE" x="23.9" y="20.3" size="1" layer="27" ratio="10" rot="R90"/>
 </element>
-<element name="CN2" library="jaw" package="HEADER-3X2-PTH" value="DO NOT PLACE" x="1.25" y="6.25" smashed="yes" rot="R270">
+<element name="CN2" library="jaw" package="HEADER-3X2-POGO" value="DO NOT PLACE" x="1.25" y="6.25" smashed="yes" rot="R270">
 <attribute name="NAME" x="1.93" y="8.495" size="1.27" layer="25" ratio="10" display="off"/>
 <attribute name="VALUE" x="-1.925" y="7.52" size="1.27" layer="27" rot="R270" display="off"/>
@@
 <wire x1="17.5" y1="14.25" x2="19.5" y2="14.25" width="0.25" layer="1"/>
 <wire x1="19.5" y1="14.25" x2="21.375" y2="16.125" width="0.25" layer="1"/>
-<via x="22.25" y="17.75" extent="1-16" drill="0.35"/>
-<via x="22.25" y="15.25" extent="1-16" drill="0.35"/>
-<via x="19.75" y="15.25" extent="1-16" drill="0.35"/>
+<via x="22" y="17.5" extent="1-16" drill="0.35"/>
+<via x="22" y="15.5" extent="1-16" drill="0.35"/>
+<via x="20" y="15.5" extent="1-16" drill="0.35"/>
 <wire x1="13.7" y1="11.05" x2="13.7" y2="12.5" width="0.25" layer="1"/>
 <wire x1="13.7" y1="12.5" x2="13.7" y2="14" width="0.25" layer="1"/>
@@
 <via x="20.75" y="31.75" extent="1-16" drill="0.35"/>
 <via x="33" y="29.95" extent="1-16" drill="0.35"/>
+<via x="20" y="17.5" extent="1-16" drill="0.35"/>
 </signal>
 <signal name="VCC">
@@
 <wire x1="12.5" y1="16.5" x2="13.4" y2="17.4" width="0.25" layer="15"/>
 <wire x1="13.4" y1="17.4" x2="17.25" y2="17.4" width="0.25" layer="15"/>
-<wire x1="17.25" y1="17.4" x2="17.65" y2="17" width="0.25" layer="15"/>
-<wire x1="17.65" y1="17" x2="23.7" y2="17" width="0.25" layer="15"/>
-<wire x1="23.7" y1="17" x2="25.05" y2="18.35" width="0.25" layer="15"/>
+<wire x1="17.25" y1="17.4" x2="17.85" y2="16.8" width="0.25" layer="15"/>
+<wire x1="17.85" y1="16.8" x2="23.5" y2="16.8" width="0.25" layer="15"/>
+<wire x1="23.5" y1="16.8" x2="25.05" y2="18.35" width="0.25" layer="15"/>
 <wire x1="25.05" y1="18.35" x2="25.05" y2="20" width="0.25" layer="15"/>
 <wire x1="9.5" y1="2.5" x2="11.95" y2="16.5" width="0" layer="19" extent="16-16"/>

Commit message: power ckt
Parts:
- removed Q2: DMP2035U-7, jaw:SOT-23
- removed R11: 1M, jaw:SMD0603
- added C3: 1u, jaw:SMD0603
- added R1: 1M, jaw:SMD0603
- added U3: AP22802A, jaw:SOT-23-5
- moved Q1 0.25 mm to (26.8, 28.5)
Connections:
- net GND: now also C3.2, R1.1, U3.2
- net NPWREN: now also R1.2, U3.4; no longer Q2.1, R11.2
- net VCC: now also C3.1, U3.5; no longer D1.C, Q2.2, R11.1, SPKR1.P1
- net VCCE: now also D1.C, SPKR1.P1, U3.1; no longer Q2.3
Routing:
- net VCCE: track 57.9 -> 67.8 mm
- net GND: track 96.9 -> 103.1 mm
- net VCC: track 36.6 -> 31.5 mm, vias 10 -> 9
- net NPWREN: track 9.26 -> 7.99 mm
- net SPIMISO: track 34.6 -> 35.2 mm
Other:
- board text added: "AMIKETO/2 Rev. 1"
- board text added: "JAW 2015-10"
- board text removed: "AMIKETO/2 Rev. 0"
- board text removed: "JAW 2015-07"

Commit message: tweak
Parts:
- added SJ1: (no value), SparkFun-Passives:PAD-JUMPER-2-NO_YES_SILK
- D1: device jaw:SOD-323 -> jaw:SMD0805D
- moved SPKR1 0.27 mm to (31.5, 25.1)
- moved C19 0.05 mm to (14.5, 11.0)
Connections:
- net NPWREN renamed PWREN
- net N$21: now also SJ1.1
- net VCC: now also SJ1.2
Routing:
- net N$21: track 24.3 -> 30.4 mm
- net VCC: track 31.5 -> 34.0 mm
- net GND: vias 42 -> 48
Other:
- board text added: "D/CS"
- board text added: "D/DC"
- board text added: "MISO"
- board text added: "MOSI"
- board text added: "NRST"
- board text added: "SCK"
- board text added: "SCL"
- board text added: "SDA"
- board text added: "VCC"
- board text removed: ""halber mensch""
