File: cad/amiketo_2hm.sch (EAGLE design)
At the start: 56 parts, among them CN1 MICROSD-EJECT, CN2 DO NOT PLACE, Q1 IRLML6344TRPBF, Q2 DMP2035U-7, SW2 SWITCHKMR211, SW3 SWITCHKMR211, U1 STM32F411/48, U2 LIS3DH, X1 12MHz, X2 32k768

Commit message: tweak
Parts:
- CN2: device jaw:HEADER-3X2-PTH -> jaw:HEADER-3X2-POGO
Changed lines of the file:
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@@
 <part name="VCCE1" library="jaw" deviceset="PWR-VCCE" device=""/>
 <part name="R11" library="jaw" deviceset="R" device="0603" value="1M"/>
-<part name="CN2" library="jaw" deviceset="HEADER-3X2" device="-PTH" value="DO NOT PLACE"/>
+<part name="CN2" library="jaw" deviceset="HEADER-3X2" device="-POGO" value="DO NOT PLACE"/>
 <part name="JP2" library="SparkFun-Connectors" deviceset="M13" device=""/>
 <part name="VCCE3" library="jaw" deviceset="PWR-VCCE" device=""/>

Commit message: power ckt
Parts:
- removed Q2: DMP2035U-7, jaw:MOSFET-P
- removed R11: 1M, jaw:R0603
- added C3: 1u, jaw:C0603
- added R1: 1M, jaw:R0603
- added U3: AP22802A, jaw:NCP380
Connections:
- net GND: now also C3.P$2, R1.P$1, U3.GND
- net NPWREN: now also R1.P$2, U3.EN; no longer Q2.G, R11.P$2
- net VCC: now also C3.P$1, U3.IN; no longer D1.C, Q2.S, R11.P$1, SPKR1.P1
- net VCCE: now also D1.C, SPKR1.P1, U3.OUT; no longer Q2.D
Changed lines of the file:
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@@
 <part name="SPKR1" library="jaw" deviceset="PUI-5040" device=""/>
 <part name="D1" library="jaw" deviceset="DIODE" device="SOD-323" value="any"/>
-<part name="VCC3" library="jaw" deviceset="PWR-VCC" device=""/>
 <part name="GND10" library="jaw" deviceset="PWR-GND" device=""/>
 <part name="Q1" library="jaw" deviceset="MOSFET" device="SOT-23" value="IRLML6344TRPBF"/>
@@
 <part name="VR1" library="jaw" deviceset="REGULATOR" device="-SOT23-3" value="mcp1700 /3v3"/>
 <part name="FRAME2" library="frames" deviceset="FRAME_B_L" device=""/>
-<part name="Q2" library="jaw" deviceset="MOSFET-P" device="" value="DMP2035U-7"/>
-<part name="VCC5" library="jaw" deviceset="PWR-VCC" device=""/>
-<part name="VCCE1" library="jaw" deviceset="PWR-VCCE" device=""/>
-<part name="R11" library="jaw" deviceset="R" device="0603" value="1M"/>
 <part name="CN2" library="jaw" deviceset="HEADER-3X2" device="-POGO" value="DO NOT PLACE"/>
 <part name="JP2" library="SparkFun-Connectors" deviceset="M13" device=""/>
@@
 <part name="U$5" library="jaw" deviceset="FIDUCIAL" device=""/>
 <part name="U$6" library="Sparkfun-Aesthetics" deviceset="FIDUCIAL" device="UFIDUCIAL"/>
+<part name="U3" library="jaw" deviceset="NCP380" device="" value="AP22802A"/>
+<part name="GND1" library="jaw" deviceset="PWR-GND" device=""/>
+<part name="VCCE5" library="jaw" deviceset="PWR-VCCE" device=""/>
+<part name="VCC4" library="jaw" deviceset="PWR-VCC" device=""/>
+<part name="C3" library="jaw" deviceset="C" device="0603" value="1u"/>
+<part name="VCC5" library="jaw" deviceset="PWR-VCC" device=""/>
+<part name="GND2" library="jaw" deviceset="PWR-GND" device=""/>
+<part name="VCCE1" library="jaw" deviceset="PWR-VCCE" device=""/>
+<part name="R1" library="jaw" deviceset="R" device="0603" value="1M"/>
 </parts>
 <sheets>
@@
 <instance part="SPKR1" gate="G$1" x="314.96" y="213.36"/>
 <instance part="D1" gate="G$1" x="304.8" y="213.36" rot="R90"/>
-<instance part="VCC3" gate="G$1" x="312.42" y="228.6"/>
 <instance part="GND10" gate="G$1" x="312.42" y="180.34"/>
 <instance part="Q1" gate="G$1" x="312.42" y="195.58"/>
@@
 <instance part="FRAME2" gate="G$1" x="0" y="0"/>
 <instance part="FRAME2" gate="G$2" x="325.12" y="0"/>
-<instance part="Q2" gate="G$1" x="226.06" y="60.96" rot="MR180"/>
-<instance part="VCC5" gate="G$1" x="226.06" y="78.74"/>
-<instance part="VCCE1" gate="G$1" x="243.84" y="60.96"/>
-<instance part="R11" gate="G$1" x="218.44" y="68.58" rot="R180"/>
 <instance part="CN2" gate="G$1" x="383.54" y="88.9"/>
 <instance part="JP2" gate="G$1" x="396.24" y="137.16" rot="R180"/>
@@
 <instance part="U$5" gate="G$1" x="419.1" y="25.4"/>
 <instance part="U$6" gate="G$1" x="414.02" y="25.4"/>
+<instance part="U3" gate="G$1" x="231.14" y="53.34"/>
+<instance part="GND1" gate="G$1" x="231.14" y="40.64"/>
+<instance part="VCCE5" gate="G$1" x="246.38" y="60.96"/>
+<instance part="VCC4" gate="G$1" x="215.9" y="60.96"/>
+<instance part="C3" gate="G$1" x="195.58" y="53.34"/>
+<instance part="VCC5" gate="G$1" x="195.58" y="60.96"/>
+<instance part="GND2" gate="G$1" x="195.58" y="48.26"/>
+<instance part="VCCE1" gate="G$1" x="312.42" y="228.6"/>
+<instance part="R1" gate="G$1" x="215.9" y="48.26" rot="R90"/>
 </instances>
 <busses>
@@
 <label x="396.24" y="93.98" size="1.27" layer="95"/>
 </segment>
+<segment>
+<pinref part="U3" gate="G$1" pin="GND"/>
+<pinref part="GND1" gate="G$1" pin="GND"/>
+<pinref part="R1" gate="G$1" pin="P$1"/>
+<wire x1="215.9" y1="43.18" x2="231.14" y2="43.18" width="0.1524" layer="91"/>
+<junction x="231.14" y="43.18"/>
+</segment>
+<segment>
+<pinref part="C3" gate="G$1" pin="P$2"/>
+<pinref part="GND2" gate="G$1" pin="GND"/>
+</segment>
 </net>
 <net name="VCC" class="0">
@@
 </segment>
 <segment>
-<pinref part="SPKR1" gate="G$1" pin="P1"/>
-<pinref part="VCC3" gate="G$1" pin="VCC"/>
-<wire x1="312.42" y1="226.06" x2="312.42" y2="223.52" width="0.1524" layer="91"/>
-<pinref part="D1" gate="G$1" pin="C"/>
-<wire x1="304.8" y1="215.9" x2="304.8" y2="223.52" width="0.1524" layer="91"/>
-<wire x1="304.8" y1="223.52" x2="312.42" y2="223.52" width="0.1524" layer="91"/>
-<junction x="312.42" y="223.52"/>
-</segment>
-<segment>
 <pinref part="R3" gate="G$1" pin="P$2"/>
 <pinref part="R9" gate="G$1" pin="P$2"/>
@@
 </segment>
 <segment>
-<pinref part="VCC5" gate="G$1" pin="VCC"/>
-<pinref part="Q2" gate="G$1" pin="S"/>
-<wire x1="226.06" y1="76.2" x2="226.06" y2="68.58" width="0.1524" layer="91"/>
-<wire x1="226.06" y1="68.58" x2="226.06" y2="66.04" width="0.1524" layer="91"/>
-<pinref part="R11" gate="G$1" pin="P$1"/>
-<wire x1="223.52" y1="68.58" x2="226.06" y2="68.58" width="0.1524" layer="91"/>
-<junction x="226.06" y="68.58"/>
-</segment>
-<segment>
 <pinref part="JP2" gate="G$1" pin="2"/>
 <wire x1="386.08" y1="149.86" x2="381" y2="149.86" width="0.1524" layer="91"/>
 <label x="375.92" y="149.86" size="1.27" layer="95"/>
+</segment>
+<segment>
+<pinref part="U3" gate="G$1" pin="IN"/>
+<pinref part="VCC4" gate="G$1" pin="VCC"/>
+</segment>
+<segment>
+<pinref part="C3" gate="G$1" pin="P$1"/>
+<pinref part="VCC5" gate="G$1" pin="VCC"/>
 </segment>
 </net>
@@
 </segment>
 <segment>
-<pinref part="VCCE1" gate="G$1" pin="VCCE"/>
-<pinref part="Q2" gate="G$1" pin="D"/>
-<wire x1="243.84" y1="58.42" x2="243.84" y2="55.88" width="0.1524" layer="91"/>
-<wire x1="243.84" y1="55.88" x2="226.06" y2="55.88" width="0.1524" layer="91"/>
-</segment>
-<segment>
 <pinref part="C14" gate="G$1" pin="P$1"/>
 <wire x1="332.74" y1="154.94" x2="317.5" y2="154.94" width="0.1524" layer="91"/>
@@
 <label x="335.28" y="132.08" size="1.27" layer="95" ratio="10"/>
 </segment>
+<segment>
+<pinref part="U3" gate="G$1" pin="OUT"/>
+<pinref part="VCCE5" gate="G$1" pin="VCCE"/>
+</segment>
+<segment>
+<pinref part="SPKR1" gate="G$1" pin="P1"/>
+<wire x1="312.42" y1="226.06" x2="312.42" y2="223.52" width="0.1524" layer="91"/>
+<pinref part="D1" gate="G$1" pin="C"/>
+<wire x1="304.8" y1="215.9" x2="304.8" y2="223.52" width="0.1524" layer="91"/>
+<wire x1="304.8" y1="223.52" x2="312.42" y2="223.52" width="0.1524" layer="91"/>
+<junction x="312.42" y="223.52"/>
+<pinref part="VCCE1" gate="G$1" pin="VCCE"/>
+</segment>
 </net>
 <net name="NPWREN" class="0">
@@
 </segment>
 <segment>
-<pinref part="Q2" gate="G$1" pin="G"/>
-<wire x1="220.98" y1="63.5" x2="213.36" y2="63.5" width="0.1524" layer="91"/>
-<wire x1="213.36" y1="63.5" x2="213.36" y2="68.58" width="0.1524" layer="91"/>
-<wire x1="213.36" y1="68.58" x2="208.28" y2="68.58" width="0.1524" layer="91"/>
-<label x="203.2" y="68.58" size="1.27" layer="95"/>
-<pinref part="R11" gate="G$1" pin="P$2"/>
-<junction x="213.36" y="68.58"/>
-</segment>
-</net>
+<pinref part="U3" gate="G$1" pin="EN"/>
+<wire x1="215.9" y1="53.34" x2="210.82" y2="53.34" width="0.1524" layer="91"/>
+<label x="205.74" y="53.34" size="1.27" layer="95" ratio="10"/>
+<pinref part="R1" gate="G$1" pin="P$2"/>
+<junction x="215.9" y="53.34"/>
+</segment>
+</net>

Commit message: tweak
Parts:
- added SJ1: JUMPER-PAD-2-NOYES_SILK, SparkFun-Passives:JUMPER-PAD-2-NOYES_SILK
- D1: device jaw:DIODESOD-323 -> jaw:DIODE-0805
Connections:
- net NPWREN renamed PWREN
- net N$21: now also SJ1.1
- net VCC: now also SJ1.2
Other:
- moved on the sheet: C16, C6, R1, U3
Changed lines of the file:
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@@
 <part name="GND9" library="jaw" deviceset="PWR-GND" device=""/>
 <part name="SPKR1" library="jaw" deviceset="PUI-5040" device=""/>
-<part name="D1" library="jaw" deviceset="DIODE" device="SOD-323" value="any"/>
+<part name="D1" library="jaw" deviceset="DIODE" device="-0805" value="any"/>
 <part name="GND10" library="jaw" deviceset="PWR-GND" device=""/>
 <part name="Q1" library="jaw" deviceset="MOSFET" device="SOT-23" value="IRLML6344TRPBF"/>
@@
 <part name="VCCE1" library="jaw" deviceset="PWR-VCCE" device=""/>
 <part name="R1" library="jaw" deviceset="R" device="0603" value="1M"/>
+<part name="SJ1" library="SparkFun-Passives" deviceset="JUMPER-PAD-2-NO" device="YES_SILK" value=""/>
+<part name="VCC3" library="jaw" deviceset="PWR-VCC" device=""/>
 </parts>
 <sheets>
@@
 <instance part="GND5" gate="G$1" x="134.62" y="152.4"/>
 <instance part="GND6" gate="G$1" x="215.9" y="144.78"/>
-<instance part="VCC2" gate="G$1" x="203.2" y="172.72"/>
-<instance part="VCCA2" gate="G$1" x="215.9" y="172.72"/>
+<instance part="VCC2" gate="G$1" x="200.66" y="172.72"/>
+<instance part="VCCA2" gate="G$1" x="210.82" y="172.72"/>
 <instance part="C10" gate="G$1" x="223.52" y="152.4"/>
 <instance part="GND7" gate="G$1" x="223.52" y="144.78"/>
@@
 <instance part="CN1" gate="G$1" x="314.96" y="66.04"/>
 <instance part="GND22" gate="G$1" x="287.02" y="53.34"/>
-<instance part="C16" gate="G$1" x="330.2" y="66.04"/>
-<instance part="GND23" gate="G$1" x="330.2" y="60.96"/>
+<instance part="C16" gate="G$1" x="261.62" y="53.34"/>
+<instance part="GND23" gate="G$1" x="261.62" y="48.26"/>
 <instance part="GND13" gate="G$1" x="332.74" y="48.26"/>
 <instance part="U$2" gate="G$1" x="424.18" y="25.4"/>
@@
 <instance part="R2" gate="G$1" x="299.72" y="193.04"/>
 <instance part="VCCE2" gate="G$1" x="287.02" y="60.96"/>
-<instance part="VCCE4" gate="G$1" x="330.2" y="73.66"/>
-<instance part="C6" gate="G$1" x="335.28" y="66.04"/>
+<instance part="VCCE4" gate="G$1" x="261.62" y="60.96"/>
+<instance part="C6" gate="G$1" x="266.7" y="53.34"/>
 <instance part="C7" gate="G$1" x="226.06" y="165.1" rot="R270"/>
 <instance part="U2" gate="G$1" x="314.96" y="134.62"/>
@@
 <instance part="U$5" gate="G$1" x="419.1" y="25.4"/>
 <instance part="U$6" gate="G$1" x="414.02" y="25.4"/>
-<instance part="U3" gate="G$1" x="231.14" y="53.34"/>
-<instance part="GND1" gate="G$1" x="231.14" y="40.64"/>
-<instance part="VCCE5" gate="G$1" x="246.38" y="60.96"/>
-<instance part="VCC4" gate="G$1" x="215.9" y="60.96"/>
+<instance part="U3" gate="G$1" x="226.06" y="53.34"/>
+<instance part="GND1" gate="G$1" x="226.06" y="40.64"/>
+<instance part="VCCE5" gate="G$1" x="241.3" y="60.96"/>
+<instance part="VCC4" gate="G$1" x="210.82" y="60.96"/>
 <instance part="C3" gate="G$1" x="195.58" y="53.34"/>
 <instance part="VCC5" gate="G$1" x="195.58" y="60.96"/>
 <instance part="GND2" gate="G$1" x="195.58" y="48.26"/>
 <instance part="VCCE1" gate="G$1" x="312.42" y="228.6"/>
-<instance part="R1" gate="G$1" x="215.9" y="48.26" rot="R90"/>
+<instance part="R1" gate="G$1" x="210.82" y="48.26" rot="R90"/>
+<instance part="SJ1" gate="G$1" x="228.6" y="175.26"/>
+<instance part="VCC3" gate="G$1" x="236.22" y="177.8"/>
 </instances>
 <busses>
@@
 <pinref part="GND23" gate="G$1" pin="GND"/>
 <pinref part="C6" gate="G$1" pin="P$2"/>
-<wire x1="335.28" y1="63.5" x2="330.2" y2="63.5" width="0.1524" layer="91"/>
-<junction x="330.2" y="63.5"/>
+<wire x1="266.7" y1="50.8" x2="261.62" y2="50.8" width="0.1524" layer="91"/>
+<junction x="261.62" y="50.8"/>
 </segment>
 <segment>
@@
 <pinref part="GND1" gate="G$1" pin="GND"/>
 <pinref part="R1" gate="G$1" pin="P$1"/>
-<wire x1="215.9" y1="43.18" x2="231.14" y2="43.18" width="0.1524" layer="91"/>
-<junction x="231.14" y="43.18"/>
+<wire x1="210.82" y1="43.18" x2="226.06" y2="43.18" width="0.1524" layer="91"/>
+<junction x="226.06" y="43.18"/>
 </segment>
 <segment>
@@
 <segment>
 <pinref part="U1" gate="G$1" pin="VCC"/>
-<wire x1="193.04" y1="167.64" x2="203.2" y2="167.64" width="0.1524" layer="91"/>
+<wire x1="193.04" y1="167.64" x2="200.66" y2="167.64" width="0.1524" layer="91"/>
 <pinref part="VCC2" gate="G$1" pin="VCC"/>
-<wire x1="203.2" y1="167.64" x2="203.2" y2="170.18" width="0.1524" layer="91"/>
+<wire x1="200.66" y1="167.64" x2="200.66" y2="170.18" width="0.1524" layer="91"/>
 </segment>
 <segment>
@@
 <pinref part="C3" gate="G$1" pin="P$1"/>
 <pinref part="VCC5" gate="G$1" pin="VCC"/>
+</segment>
+<segment>
+<pinref part="SJ1" gate="G$1" pin="2"/>
+<pinref part="VCC3" gate="G$1" pin="VCC"/>
+<wire x1="233.68" y1="175.26" x2="236.22" y2="175.26" width="0.1524" layer="91"/>
 </segment>
 </net>
@@
 <segment>
 <pinref part="U1" gate="G$1" pin="VCCA"/>
-<wire x1="193.04" y1="165.1" x2="215.9" y2="165.1" width="0.1524" layer="91"/>
+<wire x1="193.04" y1="165.1" x2="210.82" y2="165.1" width="0.1524" layer="91"/>
 <pinref part="VCCA2" gate="G$1" pin="VCCA"/>
-<wire x1="215.9" y1="165.1" x2="215.9" y2="170.18" width="0.1524" layer="91"/>
+<wire x1="210.82" y1="165.1" x2="210.82" y2="170.18" width="0.1524" layer="91"/>
 </segment>
 </net>
@@
 <wire x1="223.52" y1="165.1" x2="223.52" y2="170.18" width="0.1524" layer="91"/>
 <junction x="223.52" y="165.1"/>
+<pinref part="SJ1" gate="G$1" pin="1"/>
+<wire x1="223.52" y1="170.18" x2="223.52" y2="175.26" width="0.1524" layer="91"/>
+<junction x="223.52" y="170.18"/>
 </segment>
 </net>
@@
 <pinref part="VCCE4" gate="G$1" pin="VCCE"/>
 <pinref part="C6" gate="G$1" pin="P$1"/>
-<wire x1="335.28" y1="71.12" x2="330.2" y2="71.12" width="0.1524" layer="91"/>
-<junction x="330.2" y="71.12"/>
+<wire x1="266.7" y1="58.42" x2="261.62" y2="58.42" width="0.1524" layer="91"/>
+<junction x="261.62" y="58.42"/>
 </segment>
 <segment>
@@
 </segment>
 </net>
-<net name="NPWREN" class="0">
+<net name="PWREN" class="0">
 <segment>
 <pinref part="U1" gate="G$1" pin="PB5"/>
@@
 <segment>
 <pinref part="U3" gate="G$1" pin="EN"/>
-<wire x1="215.9" y1="53.34" x2="210.82" y2="53.34" width="0.1524" layer="91"/>
-<label x="205.74" y="53.34" size="1.27" layer="95" ratio="10"/>
+<wire x1="210.82" y1="53.34" x2="205.74" y2="53.34" width="0.1524" layer="91"/>
+<label x="203.2" y="53.34" size="1.27" layer="95" ratio="10"/>
 <pinref part="R1" gate="G$1" pin="P$2"/>
-<junction x="215.9" y="53.34"/>
-</segment>
-</net>
+<junction x="210.82" y="53.34"/>
+</segment>
+</net>
